File: pcbnew/pcad2kicadpcb_plugin/examples/CK1202_V1.kicad_pcb (KiCad board)
At the start: 6 copper layers, 280 x 228.3 mm, 332 parts

Commit message: supported stand-alone text and lines for pcad2kicad schematic conversion; updated CK1202_V1.kicad_pcb file corresponding to the previous commit
Other:
- board text added: ".467444.160r r Ver. 1"
- board text added: ".767444.161r r Ver. 1"
- board text added: "1"
- board text added: "1,5max"
- board text added: "3max"
- board text added: "5,5max"
- board text added: "8,5max"
- board text added: "FS1"
- board text added: "FS2"
- board text added: "FS3"
- board text added: "FS4"
- board text added: "IN RF"
- board text added: "IN SYNC"
- board text added: "Material : FR-4r ------------------------r Thickness of PCB: 1,5mmr ------------------------r Layers:r ------------------------r 1. Top Silk r 2. Top Mask (Solder Resist)r 3. Top (Surface plating - GOLD)r (Cu - 35mkm) , Laminate 0,3-0,4mmr 4. Power (Plane Type)r 5. INT1r 6. INT2r 7. GND (Plane Type)r 8. Bottom (Surface plating - GOLD)r 9. Bot Mask (Solder Resist)r 10. Bot Silk"
- board text added: "Max element height on bottom"
- board text added: "Or r Ur r Tr r"
- board text added: "USB 2.0"
Changed lines of the file:
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@@
     (links 1486)
     (no_connects 391)
-    (area 348.896999 -1.721514 676.8424 231.260001)
+    (area 348.896999 -1.721514 1210.651627 231.260001)
     (thickness 1.6)
     (drawings 92)
@@
     )
   )
-  (gr_text "" (at 594.71 220.576667) (layer F.Cu)
+  (gr_text ".467444.160\r\n\r\nVer. 1" (at 615.543333 220.576667) (layer F.Cu)
     (effects (font (size 2.272727 1.25) (thickness 0.25)))
   )
-  (gr_text "" (at 594.81 220.876667) (layer B.Cu)
+  (gr_text ".767444.161\r\n\r\nVer. 1" (at 615.643333 220.876667) (layer B.Cu)
     (effects (font (size 2.272727 1.25) (thickness 0.25)) (justify mirror))
   )
@@
   (gr_line (start 639.51 2.81) (end 359.51 2.81) (layer Edge.Cuts) (width 0.3))
   (gr_line (start 639.51 2.81) (end 359.51 2.81) (layer Edge.Cuts) (width 0.127))
-  (gr_text "" (at 509.21 63.202) (layer F.SilkS)
+  (gr_text 1 (at 509.814762 63.202) (layer F.SilkS)
     (effects (font (size 1.385455 0.762) (thickness 0.152)))
   )
-  (gr_text "" (at 476.91 86.402) (layer F.SilkS)
+  (gr_text 1 (at 477.514762 86.402) (layer F.SilkS)
     (effects (font (size 1.385455 0.762) (thickness 0.152)))
   )
-  (gr_text "" (at 389.69 145.823333) (layer F.SilkS)
+  (gr_text "O\r\n\r\nU\r\n\r\nT\r\n\r\n" (at 419.451905 145.823333) (layer F.SilkS)
     (effects (font (size 4.545455 2.5) (thickness 0.4)))
   )
-  (gr_text "" (at 376.77 158.056667) (layer F.SilkS)
+  (gr_text FS4 (at 379.74619 158.056667) (layer F.SilkS)
     (effects (font (size 2.272727 1.25) (thickness 0.25)))
   )
-  (gr_text "" (at 376.73 145.096667) (layer F.SilkS)
+  (gr_text FS3 (at 379.70619 145.096667) (layer F.SilkS)
     (effects (font (size 2.272727 1.25) (thickness 0.25)))
   )
-  (gr_text "" (at 376.69 122.136667) (layer F.SilkS)
+  (gr_text FS1 (at 379.66619 122.136667) (layer F.SilkS)
     (effects (font (size 2.272727 1.25) (thickness 0.25)))
   )
-  (gr_text "" (at 376.69 99.336667) (layer F.SilkS)
+  (gr_text "IN RF" (at 381.650317 99.336667) (layer F.SilkS)
     (effects (font (size 2.272727 1.25) (thickness 0.25)))
   )
-  (gr_text "" (at 376.05 45.336667) (layer F.SilkS)
+  (gr_text "IN SYNC" (at 382.994444 45.336667) (layer F.SilkS)
     (effects (font (size 2.272727 1.25) (thickness 0.25)))
   )
-  (gr_text "" (at 376.69 134.376667) (layer F.SilkS)
+  (gr_text FS2 (at 379.66619 134.376667) (layer F.SilkS)
     (effects (font (size 2.272727 1.25) (thickness 0.25)))
   )
-  (gr_text "" (at 386.05 182.136667) (layer F.SilkS)
+  (gr_text "USB 2.0" (at 392.994444 182.136667) (layer F.SilkS)
     (effects (font (size 2.272727 1.25) (thickness 0.25)))
   )
-  (gr_text "" (at 676.69 120.403933) (layer Dwgs.User)
+  (gr_text "Material : FR-4\r\n------------------------\r\nThickness of PCB: 1,5mm\r\n------------------------\r\nLayers:\r\n------------------------\r\n1. Top Silk \r\n2. Top Mask (Solder Resist)\r\n3. Top (Surface plating - GOLD)\r\n(Cu - 35mkm) , Laminate 0,3-0,4mm\r\n4. Power (Plane Type)\r\n5. INT1\r\n6. INT2\r\n7. GND (Plane Type)\r\n8. Bottom (Surface plating - GOLD)\r\n9. Bot Mask (Solder Resist)\r\n10. Bot Silk" (at 1184.760556 120.403933) (layer Dwgs.User)
     (effects (font (size 3.071091 1.6891) (thickness 0.3048)))
   )
@@
   (gr_line (start 364.01 5.86) (end 365.01 5.86) (layer Dwgs.User) (width 0.1))
   (gr_line (start 364.51 5.36) (end 364.51 6.36) (layer Dwgs.User) (width 0.1))
-  (gr_text "" (at 373.71 227.176667) (layer Dwgs.User)
+  (gr_text 1,5max (at 377.519524 227.176667) (layer Dwgs.User)
     (effects (font (size 1.454545 0.8) (thickness 0.12)))
   )
@@
   (gr_line (start 363.91 99.01) (end 362.51 99.01) (layer Dwgs.User) (width 0.254))
   (gr_line (start 364.01 44.81) (end 362.51 44.81) (layer Dwgs.User) (width 0.254))
-  (gr_text "" (at 373.51 5.776667) (layer Dwgs.User)
+  (gr_text 1,5max (at 377.319524 5.776667) (layer Dwgs.User)
     (effects (font (size 1.454545 0.8) (thickness 0.12)))
   )
@@
   (gr_line (start 500.51 5.36) (end 500.51 6.36) (layer Dwgs.User) (width 0.1))
   (gr_line (start 500.01 5.86) (end 501.01 5.86) (layer Dwgs.User) (width 0.1))
-  (gr_text "" (at 529.51 227.176667) (layer Dwgs.User)
+  (gr_text 5,5max (at 533.319524 227.176667) (layer Dwgs.User)
     (effects (font (size 1.454545 0.8) (thickness 0.12)))
   )
-  (gr_text "" (at 529.61 220.176667) (layer Dwgs.User)
+  (gr_text 3max (at 532.149683 220.176667) (layer Dwgs.User)
     (effects (font (size 1.454545 0.8) (thickness 0.12)))
   )
-  (gr_text "" (at 529.41 214.576667) (layer Dwgs.User)
+  (gr_text 8,5max (at 533.219524 214.576667) (layer Dwgs.User)
     (effects (font (size 1.454545 0.8) (thickness 0.12)))
   )
-  (gr_text "" (at 529.51 12.976667) (layer Dwgs.User)
+  (gr_text 3max (at 532.049683 12.976667) (layer Dwgs.User)
     (effects (font (size 1.454545 0.8) (thickness 0.12)))
   )
-  (gr_text "" (at 529.81 5.976667) (layer Dwgs.User)
+  (gr_text 5,5max (at 533.619524 5.976667) (layer Dwgs.User)
     (effects (font (size 1.454545 0.8) (thickness 0.12)))
   )
   (gr_line (start 622.51 224.11) (end 622.51 231.11) (layer Dwgs.User) (width 0.1))
-  (gr_text "" (at 629.01 182.676667) (layer Dwgs.User)
+  (gr_text 1,5max (at 632.819524 182.676667) (layer Dwgs.User)
     (effects (font (size 1.454545 0.8) (thickness 0.12)))
   )
-  (gr_text "" (at 628.01 5.876667) (layer Dwgs.User)
+  (gr_text 1,5max (at 631.819524 5.876667) (layer Dwgs.User)
     (effects (font (size 1.454545 0.8) (thickness 0.12)))
   )
-  (gr_text "" (at 620.01 -0.523333) (layer Dwgs.User)
+  (gr_text "Max element height on bottom" (at 637.787778 -0.523333) (layer Dwgs.User)
     (effects (font (size 1.454545 0.8) (thickness 0.12)))
   )
   (gr_line (start 622.51 2.81) (end 622.51 9.81) (layer Dwgs.User) (width 0.1))
   (gr_line (start 359.51 2.81) (end 364.01 2.81) (layer Dwgs.User) (width 0.25))
-  (gr_text "" (at 509.71 227.176667) (layer Dwgs.User)
+  (gr_text 1,5max (at 513.519524 227.176667) (layer Dwgs.User)
     (effects (font (size 1.454545 0.8) (thickness 0.12)))
   )
-  (gr_text "" (at 509.51 5.776667) (layer Dwgs.User)
+  (gr_text 1,5max (at 513.319524 5.776667) (layer Dwgs.User)
     (effects (font (size 1.454545 0.8) (thickness 0.12)))
   )

Commit message: pcad2kicadpcb: fixed an issue with setting the Reference and Value of a module
Parts:
- 1, 10, 11, 12, 13, 2, 4, 5, 6, 7, 8, 9: value (none) -> YESF-085/50
- 3, TP1, TP10, TP11, TP12, TP13, TP14, TP15, TP16, TP17, TP18, TP19, TP2, TP20, TP21, TP22, TP23, TP24, TP25, TP26, TP27, TP3, TP4, TP5, TP6, TP7, TP8, TP9: value (none) -> PIN40X40X24
- C1, C2, C28: value (none) -> 1000
- C10, C100, C101, C102, C103, C104, C105, C106, C107, C108, C109, C110, C112, C113, C114, C115, C116, C117, C118, C119, C12, C120, C121, C122, C123, C13, C14, C15, C16, C17, C20, C23, C24, C30, C32, C33, C38, C39, C40, C41, C46, C47, C48, C49, C50, C51, C52, C53, C54, C55, C56, C58, C60, C61, C62, C63, C64, C68, C69, C7, C70, C72, C75, C78, C79, C8, C82, C83, C85, C86, C89, C9, C90, C91, C92, C93, C94, C96, C97, C98, C99: value (none) -> 0,1 мк
- C11, C18, C21, C26, C27, C29, C31, C34, C35, C36, C37, C42, C43, C44, C45, C57, C59, C66, C67, C74, C76, C77, C81, C87, C88, C95: value (none) -> 10 мк
- C111, C19, C6, C84: value (none) -> 0,01 мк
- C22, C25, C71, C73, C80, R36, R44, R45, R59, R63: value (none) -> 100
- C3: value (none) -> 0,022 мкФ
- C4: value (none) -> 680
- C5: value (none) -> 47
- C65: value (none) -> 220
- D1, D10, D11, D12, D13, D19, D2, D3, D5, D6: value (none) -> SN74AC245DB
- D14: value (none) -> EP2C20F484C7
- D15, D21, D26, D7, D8: value (none) -> LM1117DTX-3,3
- D16: value (none) -> LM1117DTX-ADJ
- D17, D18: value (none) -> IS61LV51216
- D20: value (none) -> EPM1270F256C4
- D22, D23: value (none) -> M25P64V6MF
- D24: value (none) -> ADSP_BF533SBB500
- D25: value (none) -> MT48LC16M16A2
- D27: value (none) -> KXO-97- 60.000 MHz
- D28: value (none) -> KXO-75- 10.000 MHz
- D29: value (none) -> LM1117-2,5
- D30, D31: value (none) -> MC100LVEL22D
- D32: value (none) -> NET2272
- D33: value (none) -> MC100LVELT23
- D34: value (none) -> FT-245RL
- D35: value (none) -> ADM705AN
- D4: value (none) -> ADF4360-8BCP
- D9: value (none) -> AD8009AR
- HL1, HL3, HL5, HL6, HL8: value (none) -> L-C170 gct
- HL2, HL4, HL7, HL9: value (none) -> L-C170 srct
- L1, L2: value (none) -> 68 нГ
- L10, L11, L12, L13, L3, L6, L7, L8, L9: value (none) -> 10 мкГ
- L14, L15: value (none) -> 1 мкГ
- L16, L17: value (none) -> 42 Ом
- L4, L5: value (none) -> 56 нГ
- R1, R13, R14, R15, R18, R2, R22, R24, R26, R3, R31, R32, R33, R34, R35, R37, R39, R46, R49, R5, R50, R57, R58, R60, R61, R62, R64, R9: value (none) -> 2,2 к
- R10, R8: value (none) -> 470
- R11: value (none) -> 6,8 к
- R12, R80: value (none) -> 4,7 к
- R16, R17, R19, R81: value (none) -> 10 к
- R20, R21, R23, R25: value (none) -> 1,2 к
- R27, R28, R29, R30, R4, R7: value (none) -> 51
- R38, R47, R48: value (none) -> 2,2k
- R40, R41, R42, R43, R51, R52, R53, R54: value (none) -> 510
- R55, R56: value (none) -> 0
- R6: value (none) -> 15 к
- R65: value (none) -> 1 к
- R66: value (none) -> 2,43 к
- R67, R68, R69, R70, R79: value (none) -> 1,5 к
- R71, R72, R73, R74: value (none) -> 820
- R75: value (none) -> 33
- R76: value (none) -> 47 к
- R77, R78: value (none) -> 39,2
- R82: value (none) -> 1 М
- R83, R84: value (none) -> 2,2K
- U1, U2: value (none) -> FDS9431A
- VD1, VD2: value (none) -> ZHCS1000
- VD3: value (none) -> 2D522B
- X1: value (none) -> URB-1001
- XP1, XP2, XP6: value (none) -> XP-JP
- XP3: value (none) -> BH2-10
- XP4: value (none) -> BH10R
- XP5: value (none) -> BH-14
- XP7, XP8: value (none) -> DIN EN 60603 121 A 10139 X
- XW1, XW2, XW3, XW4, XW5, XW6: value (none) -> C340-022D
