File: demos/microwave/microwave.kicad_pcb (KiCad board)
At the start: 2 copper layers, 4 parts

Commit message: Update old demo board files. Minor code cleaning.
Other:
- board outline added: 292.1 x 120.7 mm
Changed lines of the file:
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@@
     (15 Dessus.Cu signal)
     (0 Dessous.Cu signal)
-    (16 Dessous.Adhes user)
-    (17 Dessus.Adhes user)
-    (18 Dessous.Pate user)
-    (19 Dessus.Pate user)
-    (20 Dessous.SilkS user)
-    (21 Dessus.SilkS user)
-    (22 Dessous.Masque user)
-    (23 Dessus.Masque user)
-    (24 Dessin.User user)
+    (16 B.Adhes user)
+    (17 F.Adhes user)
+    (18 B.Paste user)
+    (19 F.Paste user)
+    (20 B.SilkS user)
+    (21 F.SilkS user)
+    (22 B.Mask user)
+    (23 F.Mask user)
+    (24 Dwgs.User user)
     (25 Cmts.User user)
     (26 Eco1.User user)
     (27 Eco2.User user)
-    (28 Contours.Ci user)
-  )
+    (28 Edge.Cuts user)
+   )
   (setup
     (last_trace_width 0.254)
@@
   (module POLY (layer Dessus.Cu)
     (at 203.2 144.78)
-    (fp_text reference POLY (at 0 0.0762) (layer Dessus.SilkS)
+    (fp_text reference POLY (at 0 0.0762) (layer F.SilkS)
       (effects (font (size 0.0762 0.0762) (thickness 0.2032)))
     )
-    (fp_text value VAL** (at 0 -0.0762) (layer Dessus.SilkS)
+    (fp_text value VAL** (at 0 -0.0762) (layer F.SilkS)
       (effects (font (size 0.0762 0.0762) (thickness 0.2032)))
     )
@@
   (module POLY (layer Dessus.Cu)
     (at 203.17968 117.21084)
-    (fp_text reference POLY (at 0 0.0762) (layer Dessus.SilkS)
+    (fp_text reference POLY (at 0 0.0762) (layer F.SilkS)
       (effects (font (size 0.0762 0.0762) (thickness 0.2032)))
     )
-    (fp_text value VAL** (at 0 -0.0762) (layer Dessus.SilkS)
+    (fp_text value VAL** (at 0 -0.0762) (layer F.SilkS)
       (effects (font (size 0.0762 0.0762) (thickness 0.2032)))
     )
@@
   (module POLY (layer Dessus.Cu)
     (at 203.2 119.38)
-    (fp_text reference POLY (at 0 0.0762) (layer Dessus.SilkS)
+    (fp_text reference POLY (at 0 0.0762) (layer F.SilkS)
       (effects (font (size 0.0762 0.0762) (thickness 0.2032)))
     )
-    (fp_text value VAL** (at 0 -0.0762) (layer Dessus.SilkS)
+    (fp_text value VAL** (at 0 -0.0762) (layer F.SilkS)
       (effects (font (size 0.0762 0.0762) (thickness 0.2032)))
     )
@@
   (module POLY (layer Dessus.Cu)
     (at 203.18984 121.54408)
-    (fp_text reference POLY (at 0 0.0762) (layer Dessus.SilkS)
+    (fp_text reference POLY (at 0 0.0762) (layer F.SilkS)
       (effects (font (size 0.0762 0.0762) (thickness 0.2032)))
     )
-    (fp_text value VAL** (at 0 -0.0762) (layer Dessus.SilkS)
+    (fp_text value VAL** (at 0 -0.0762) (layer F.SilkS)
       (effects (font (size 0.0762 0.0762) (thickness 0.2032)))
     )
@@
     )
   )
-  (gr_line (start 203.50988 120.54332) (end 203.50988 120.55348) (angle 90) (layer Dessin.User) (width 0.3048))
-  (gr_line (start 202.84694 120.54332) (end 203.50988 120.54332) (angle 90) (layer Dessin.User) (width 0.3048))
-  (gr_line (start 162.4076 120.38076) (end 164.10178 120.38076) (angle 90) (layer Dessin.User) (width 0.3048))
-  (gr_line (start 59.69 201.93) (end 59.69 81.28) (angle 90) (layer Contours.Ci) (width 0.3048))
-  (gr_line (start 351.79 201.93) (end 59.69 201.93) (angle 90) (layer Contours.Ci) (width 0.3048))
-  (gr_line (start 351.79 81.28) (end 351.79 201.93) (angle 90) (layer Contours.Ci) (width 0.3048))
-  (gr_line (start 59.69 81.28) (end 351.79 81.28) (angle 90) (layer Contours.Ci) (width 0.3048))
+  (gr_line (start 203.50988 120.54332) (end 203.50988 120.55348) (angle 90) (layer Dwgs.User) (width 0.3048))
+  (gr_line (start 202.84694 120.54332) (end 203.50988 120.54332) (angle 90) (layer Dwgs.User) (width 0.3048))
+  (gr_line (start 162.4076 120.38076) (end 164.10178 120.38076) (angle 90) (layer Dwgs.User) (width 0.3048))
+  (gr_line (start 59.69 201.93) (end 59.69 81.28) (angle 90) (layer Edge.Cuts) (width 0.3048))
+  (gr_line (start 351.79 201.93) (end 59.69 201.93) (angle 90) (layer Edge.Cuts) (width 0.3048))
+  (gr_line (start 351.79 81.28) (end 351.79 201.93) (angle 90) (layer Edge.Cuts) (width 0.3048))
+  (gr_line (start 59.69 81.28) (end 351.79 81.28) (angle 90) (layer Edge.Cuts) (width 0.3048))
 )
