File: demos/kit-dev-coldfire-xilinx_5213/kit-dev-coldfire-xilinx_5213.kicad_pcb (KiCad board)
At the start: 4 copper layers, 157.5 x 91.4 mm, 162 parts, among them J1 JACK_2P, P1 CONN_6, P3 CONN_2X2, P4 CONN_20X2, Q1 3906, SW1 SW_PUSH, SW2 SW_PUSH, U1 MCF5213-LQFP100, U2 74AHC1G14, U3 MAX202, U4 74HC125, U5 MAX202, U7 PCA82C251, U8 MAX202, U9 XCR3256-TQ144, Y1 8MHz

Commit message: Very minor fixes.
Routing:
- added copper zone on VDD_layer, net VDD
- removed copper zone on 3.3V_layer, net +3.3V
