File: demos/kit-dev-coldfire-xilinx_5213/kit-dev-coldfire-xilinx_5213.kicad_pcb (KiCad board)
At the start: 4 copper layers, 157.5 x 91.4 mm, 162 parts, among them J1 JACK_2P, P1 CONN_6, P3 CONN_2X2, P4 CONN_20X2, Q1 3906, SW1 SW_PUSH, SW2 SW_PUSH, U1 MCF5213-LQFP100, U2 74AHC1G14, U3 MAX202, U4 74HC125, U5 MAX202, U7 PCA82C251, U8 MAX202, U9 XCR3256-TQ144, Y1 8MHz

Commit message: merge from production git:e53c3af 21.04.2017
Connections:
- net VDD renamed +3.3V
- BDM_PORT1 pad 1: (no net) -> Net-(BDM_PORT1-Pad1)
- BDM_PORT1 pad 21: (no net) -> Net-(BDM_PORT1-Pad21)
- BDM_PORT1 pad 22: (no net) -> Net-(BDM_PORT1-Pad22)
- SW_ONOFF1 pad 1: (no net) -> Net-(SW_ONOFF1-Pad1)
- U9 pad 102: (no net) -> Net-(U9-Pad102)
- U9 pad 103: (no net) -> Net-(U9-Pad103)
- U9 pad 106: (no net) -> Net-(U9-Pad106)
- U9 pad 110: (no net) -> Net-(U9-Pad110)
- U9 pad 120: (no net) -> Net-(U9-Pad120)
- U9 pad 121: (no net) -> Net-(U9-Pad121)
- U9 pad 133: (no net) -> Net-(U9-Pad133)
- U9 pad 14: (no net) -> Net-(U9-Pad14)
- U9 pad 141: (no net) -> Net-(U9-Pad141)
- U9 pad 15: (no net) -> Net-(U9-Pad15)
- U9 pad 16: (no net) -> Net-(U9-Pad16)
- U9 pad 18: (no net) -> Net-(U9-Pad18)
- U9 pad 19: (no net) -> Net-(U9-Pad19)
- U9 pad 21: (no net) -> Net-(U9-Pad21)
- U9 pad 22: (no net) -> Net-(U9-Pad22)
- U9 pad 23: (no net) -> Net-(U9-Pad23)
- U9 pad 25: (no net) -> Net-(U9-Pad25)
- U9 pad 26: (no net) -> Net-(U9-Pad26)
- U9 pad 29: (no net) -> Net-(U9-Pad29)
- U9 pad 30: (no net) -> Net-(U9-Pad30)
- U9 pad 34: (no net) -> Net-(U9-Pad34)
- U9 pad 35: (no net) -> Net-(U9-Pad35)
- U9 pad 36: (no net) -> Net-(U9-Pad36)
- U9 pad 37: (no net) -> Net-(U9-Pad37)
- U9 pad 38: (no net) -> Net-(U9-Pad38)
- U9 pad 39: (no net) -> Net-(U9-Pad39)
- U9 pad 40: (no net) -> Net-(U9-Pad40)
- U9 pad 41: (no net) -> Net-(U9-Pad41)
- U9 pad 55: (no net) -> Net-(U9-Pad55)
- U9 pad 56: (no net) -> Net-(U9-Pad56)
- U9 pad 60: (no net) -> Net-(U9-Pad60)
- U9 pad 61: (no net) -> Net-(U9-Pad61)
- U9 pad 62: (no net) -> Net-(U9-Pad62)
- U9 pad 63: (no net) -> Net-(U9-Pad63)
- U9 pad 65: (no net) -> Net-(U9-Pad65)
- U9 pad 66: (no net) -> Net-(U9-Pad66)
- U9 pad 67: (no net) -> Net-(U9-Pad67)
- U9 pad 68: (no net) -> Net-(U9-Pad68)
- U9 pad 69: (no net) -> Net-(U9-Pad69)
- U9 pad 70: (no net) -> Net-(U9-Pad70)
- U9 pad 71: (no net) -> Net-(U9-Pad71)
- U9 pad 72: (no net) -> Net-(U9-Pad72)
- U9 pad 74: (no net) -> Net-(U9-Pad74)
- U9 pad 75: (no net) -> Net-(U9-Pad75)
- U9 pad 77: (no net) -> Net-(U9-Pad77)
- U9 pad 78: (no net) -> Net-(U9-Pad78)
- U9 pad 79: (no net) -> Net-(U9-Pad79)
- U9 pad 80: (no net) -> Net-(U9-Pad80)
- U9 pad 81: (no net) -> Net-(U9-Pad81)
- U9 pad 82: (no net) -> Net-(U9-Pad82)
- U9 pad 83: (no net) -> Net-(U9-Pad83)
- U9 pad 84: (no net) -> Net-(U9-Pad84)
- U9 pad 86: (no net) -> Net-(U9-Pad86)
- U9 pad 87: (no net) -> Net-(U9-Pad87)
- U9 pad 88: (no net) -> Net-(U9-Pad88)
- U9 pad 9: (no net) -> Net-(U9-Pad9)
- U9 pad 90: (no net) -> Net-(U9-Pad90)
- U9 pad 91: (no net) -> Net-(U9-Pad91)
- U9 pad 92: (no net) -> Net-(U9-Pad92)
- U9 pad 93: (no net) -> Net-(U9-Pad93)
- U9 pad 94: (no net) -> Net-(U9-Pad94)
- UARTCAN0 pad 9: (no net) -> Net-(UARTCAN0-Pad9)
- UARTCAN1 pad 9: (no net) -> Net-(UARTCAN1-Pad9)
- UARTCAN2 pad 9: (no net) -> Net-(UARTCAN2-Pad9)
- VR1 pad 4: (no net) -> Net-(VR1-Pad4)
