File: demos/video/video.kicad_pcb (KiCad board)
At the start: 4 copper layers, 189 parts, among them J4 DB9FEM, P1 BNC, P10 CONN_1, P11 CONN_1, P12 CONN_1, P2 BNC, P3 BNC, P4 CONN_2, P5 CONN_5, P8 BNC, P9 CONN_1, Q1 BC848, Q2 BC848, Q3 BC848, U1 24C16, U10 BT812, U11 S5933_PQ160, U12 SIM4X32, U13 SIM4X32, U14 SIM4X32, U15 SIM4X32, U16 SIM4X32, U17 SIM4X32, U18 SIM4X32, U19 SIM4X32, U2 4C4001, U20 TDA8501, U21 XC1736APD8, U22 XC4003-VQ100, U23 XC4003/PQ100, U24 XC4005-PQ160, U3 74LS245, U4 74LS245, U5 74LS245, U6 74LS245, U7 AV9173, U8 BT253, U9 BT473, X1 10MHz, X2 30MHz, X3 4,433618MH

Commit message: Very minor fixes. *.kicad_pcb files update to current Pcbnew version.
Other:
- board outline added: 312 x 106.7 mm

Commit message: Pcbnew: Minor fix in hotkeys. Demos: add an example to use  a local fp-lib-table and local libs, and update schematics and boards.
Parts:
- BUS1: footprint BUSPCI -> connect:BUSPCI
- C1, C10, C11, C12, C13, C14, C15, C16, C17, C18, C19, C2, C20, C21, C22, C23, C24, C25, C26, C27, C28, C29, C3, C30, C31, C32, C33, C34, C35, C36, C37, C4, C43, C44, C45, C46, C47, C48, C5, C52, C53, C54, C58, C59, C6, C60, C61, C65, C66, C67, C68, C69, C7, C70, C71, C72, C73, C8, C9, R1, R10, R11, R12, R13, R14, R15, R16, R17, R18, R19, R2, R20, R21, R22, R23, R24, R25, R26, R27, R28, R29, R3, R30, R31, R32, R33, R34, R35, R36, R37, R38, R39, R4, R40, R41, R42, R43, R44, R45, R46, R47, R48, R5, R6, R7, R8, R9: footprint SM1206 -> lib_smd:SM1206
- C38, C56: footprint SM1812L -> lib_smd:SM1812L
- C39, C40, C41, C42, C51, C55, C57, C62, C63, C64: footprint SM1210L -> lib_smd:SM1210L
- C49, C50: footprint C1 -> discret:C1
- CV1: footprint CV3-30PF -> discret:CV3-30PF
- D1, D2, D3, D4: footprint D3 -> discret:D3
- D6: footprint LEDV -> discret:LEDV
- J4: footprint DB9FC -> connect:DB9FC
- L1, L2, L3, L4, L5: footprint SM1812 -> lib_smd:SM1812
- L6: footprint LRTDK -> footprints:LRTDK
- P1, P2, P3, P8: footprint SUBCLICK -> discret:SUBCLICK
- P10, P11, P9: footprint PINTST -> connect:PINTST
- P12: footprint TESTPOINT -> connect:TESTPOINT
- P4: footprint SIL-2 -> connect:SIL-2
- P5: footprint PIN_ARRAY_5x1 -> pin_array:PIN_ARRAY_5x1
- POT1: footprint POT_CMS -> lib_smd:POT_CMS
- Q1, Q2, Q3: footprint SOT23EBC -> lib_smd:SOT23EBC
- RR1, RR2, RR3, RR6, RR8: footprint SIL-9 -> connect:SIL-9
- RR4, RR5, RR7: footprint r_pack8 -> discret:r_pack8
- U1, U21: footprint 8dip300 -> dip_sockets:DIP-8__300
- U10, U11, U24: footprint PQFP160 -> lib_smd:PQFP160
- U12, U13, U14, U15, U16, U17, U18, U19: footprint SIM72 -> footprints:sim72
- U2: footprint SO28 -> lib_smd:SO28
- U20: footprint SO24E -> lib_smd:SO24E
- U22: footprint VQFP100 -> lib_smd:VQFP100
- U23: footprint PQFP100 -> lib_smd:PQFP100
- U3, U4, U5, U6: footprint SO20L -> lib_smd:SO20L
- U7: footprint SO8E -> lib_smd:SO8E
- U8: footprint PLCC84 -> footprints:PLCC84
- U9: footprint PLCC68 -> footprints:PLCC68
- W1: footprint SM1206 -> connect:GS2
- W2, W3: footprint C1 -> connect:GS2
- W4, W5: footprint C1 -> pin_array:PIN_ARRAY_2X1
- X1, X2: footprint HC-18UV -> discret:HC-18UV
- X3: footprint HC-18UH -> discret:HC-18UH
- moved J4 1.33 mm to (69.2, 138.7)
- moved W1 1.02 mm to (162.7, 132.1), turned to 90 degrees
Connections:
- net +5V renamed VCC
- net /graphic/ADR2 renamed /buspci.sch/ADR2
- net /graphic/ADR3 renamed /buspci.sch/ADR3
- net /graphic/ADR4 renamed /buspci.sch/ADR4
- net /graphic/ADR5 renamed /buspci.sch/ADR5
- net /graphic/BE-0 renamed /buspci.sch/BE-0
- net /graphic/BE-1 renamed /buspci.sch/BE-1
- net /graphic/BE-2 renamed /buspci.sch/BE-2
- net /graphic/BE-3 renamed /buspci.sch/BE-3
- net /graphic/BLANK- renamed /ESVIDEO-RVB/BLANK-
- net /graphic/CAS1- renamed /RAMS/CAS1-
- net /graphic/CLAMP renamed /ESVIDEO-RVB/CLAMP
- net /graphic/CSYNCIN- renamed /ESVIDEO-RVB/CSYNCIN-
- net /graphic/IRQ- renamed /buspci.sch/IRQ-
- net /graphic/PCA1 renamed /ESVIDEO-RVB/PCA1
- net /graphic/PTADR- renamed /buspci.sch/PTADR-
- net /graphic/PTBE-0 renamed /buspci.sch/PTBE-0
- net /graphic/PTBE-2 renamed /buspci.sch/PTBE-2
- net /graphic/PTBE-3 renamed /buspci.sch/PTBE-3
- net /graphic/PTBURST- renamed /buspci.sch/PTBURST-
- net /graphic/PTNUM1 renamed /buspci.sch/PTNUM1
- net /graphic/PTWR renamed /buspci.sch/PTWR
- net /graphic/RAS0- renamed /RAMS/RAS0-
- net /graphic/RAS1- renamed /RAMS/RAS1-
- net /graphic/RAS2- renamed /RAMS/RAS2-
- net /graphic/RAS4- renamed /RAMS/RAS4-
- net /graphic/RAS6- renamed /RAMS/RAS6-
- net /graphic/RAS7- renamed /RAMS/RAS7-
- net /graphic/RD- renamed /buspci.sch/RD-
- net /graphic/RDCAD- renamed /ESVIDEO-RVB/RDCAD-
- net /graphic/RDEMPTY renamed /buspci.sch/RDEMPTY
- net /graphic/SELECT- renamed /buspci.sch/SELECT-
- net /graphic/TVI0 renamed /ESVIDEO-RVB/TVI0
- net /graphic/TVI1 renamed /ESVIDEO-RVB/TVI1
- net /graphic/WR- renamed /buspci.sch/WR-
- net /graphic/WRCAD- renamed /ESVIDEO-RVB/WRCAD-
- net /graphic/WRCDA- renamed /ESVIDEO-RVB/WRCDA-
- net /modul/CSYNC-OUT renamed /graphic/CSYNC-OUT
- net /muxdata/ACCES_RAM- renamed /graphic/ACCES_RAM-
- net /muxdata/ACQ_ON renamed /graphic/ACQ_ON
- net /muxdata/DPC3 renamed /ESVIDEO-RVB/DPC3
- net /muxdata/DPC6 renamed /ESVIDEO-RVB/DPC6
- net /muxdata/TVB0 renamed /ESVIDEO-RVB/TVB0
- net /muxdata/TVB1 renamed /ESVIDEO-RVB/TVB1
- net /muxdata/TVB4 renamed /ESVIDEO-RVB/TVB4
- net /muxdata/TVG6 renamed /ESVIDEO-RVB/TVG6
- net /muxdata/TVG7 renamed /ESVIDEO-RVB/TVG7
- net /muxdata/X_DONE renamed /graphic/X_DONE
- net /pal-ntsc.sch/F_PALIN renamed /graphic/F_PALIN
- net /pal-ntsc.sch/HD_PAL- renamed /graphic/HD_PAL-
- net /pal-ntsc.sch/OE_PAL- renamed /ESVIDEO-RVB/OE_PAL-
- net /pal-ntsc.sch/RED_IN renamed /ESVIDEO-RVB/RED_IN
- net /pal-ntsc.sch/TVB5 renamed /ESVIDEO-RVB/TVB5
- net /pal-ntsc.sch/TVB6 renamed /ESVIDEO-RVB/TVB6
- net /pal-ntsc.sch/TVB7 renamed /ESVIDEO-RVB/TVB7
- net /pal-ntsc.sch/TVR3 renamed /ESVIDEO-RVB/TVR3
- net /pal-ntsc.sch/TVR4 renamed /ESVIDEO-RVB/TVR4
- net /pal-ntsc.sch/VD_PAL- renamed /graphic/VD_PAL-
- BUS1 pad A1: (no net) -> Net-(BUS1-PadA1)
- BUS1 pad A11: (no net) -> Net-(BUS1-PadA11)
- BUS1 pad A14: (no net) -> Net-(BUS1-PadA14)
- BUS1 pad A19: (no net) -> Net-(BUS1-PadA19)
- BUS1 pad A3: (no net) -> Net-(BUS1-PadA3)
- BUS1 pad A40: (no net) -> Net-(BUS1-PadA40)
- BUS1 pad A41: (no net) -> Net-(BUS1-PadA41)
- BUS1 pad A60: (no net) -> Net-(BUS1-PadA60)
- BUS1 pad A7: (no net) -> Net-(BUS1-PadA7)
- BUS1 pad A9: (no net) -> Net-(BUS1-PadA9)
- BUS1 pad B1: (no net) -> Net-(BUS1-PadB1)
- BUS1 pad B10: (no net) -> Net-(BUS1-PadB10)
- BUS1 pad B14: (no net) -> Net-(BUS1-PadB14)
- BUS1 pad B2: (no net) -> Net-(BUS1-PadB2)
- BUS1 pad B60: (no net) -> Net-(BUS1-PadB60)
- BUS1 pad B7: (no net) -> Net-(BUS1-PadB7)
- BUS1 pad B8: (no net) -> Net-(BUS1-PadB8)
Routing:
- net /ESVIDEO-RVB/GREEN: track 352.5 -> 355.5 mm
- net Net-(BUS1-PadB8): track 0.00 -> 2.67 mm
- net Net-(BUS1-PadB7): track 0.00 -> 2.67 mm
- net Net-(BUS1-PadB60): track 0.00 -> 2.67 mm
- net Net-(BUS1-PadB2): track 0.00 -> 2.67 mm
- net Net-(BUS1-PadB14): track 0.00 -> 2.67 mm
- net Net-(BUS1-PadB10): track 0.00 -> 2.67 mm
- net Net-(BUS1-PadB1): track 0.00 -> 2.67 mm
- net Net-(BUS1-PadA9): track 0.00 -> 2.67 mm
- net Net-(BUS1-PadA7): track 0.00 -> 2.67 mm
- net Net-(BUS1-PadA60): track 0.00 -> 2.67 mm
- net Net-(BUS1-PadA41): track 0.00 -> 2.67 mm
- net Net-(BUS1-PadA40): track 0.00 -> 2.67 mm
- net Net-(BUS1-PadA3): track 0.00 -> 2.67 mm
- net Net-(BUS1-PadA19): track 0.00 -> 2.67 mm
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- added copper zone on GND_layer, net GND
- added copper zone on VCC_layer, net VCC
- removed copper zone on Interne_1, net GND
