File: demos/video/video.kicad_pcb (KiCad board)
At the start: 4 copper layers, 312 x 106.7 mm, 189 parts, among them J4 DB9FEM, P1 BNC, P10 CONN_1, P11 CONN_1, P12 CONN_1, P2 BNC, P3 BNC, P4 CONN_2, P5 CONN_5, P8 BNC, P9 CONN_1, Q1 BC848, Q2 BC848, Q3 BC848, U1 24C16, U10 BT812, U11 S5933_PQ160, U12 SIM4X32, U13 SIM4X32, U14 SIM4X32, U15 SIM4X32, U16 SIM4X32, U17 SIM4X32, U18 SIM4X32, U19 SIM4X32, U2 4C4001, U20 TDA8501, U21 XC1736APD8, U22 XC4003-VQ100, U23 XC4003/PQ100, U24 XC4005-PQ160, U3 74LS245, U4 74LS245, U5 74LS245, U6 74LS245, U7 AV9173, U8 BT253, U9 BT473, X1 10MHz, X2 30MHz, X3 4,433618MH

Commit message: merge from production git:e53c3af 21.04.2017
Parts:
- BUS1: footprint connect:BUSPCI -> Connectors:BUSPCI
- C42: value 2,2uF -> 2.2uF
- C49, C50: footprint discret:C1 -> Discret:C1
- C54, C55, C56, C57: value 4,7uF -> 4.7uF
- CV1: footprint discret:CV3-30PF -> Discret:CV3-30PF
- D1, D2, D3, D4: footprint discret:D3 -> Discret:D3
- D6: footprint discret:LEDV -> Discret:LEDV
- J4: footprint connect:DB9FC -> Connectors:DB9FC
- L6: value 470nS -> 470ns
- P1, P2, P3, P8: footprint discret:SUBCLICK -> Discret:SUBCLICK
- P10, P11, P9: footprint connect:PINTST -> Connectors:PINTST
- P12: footprint connect:TESTPOINT -> Connectors:TESTPOINT
- P4: footprint connect:SIL-2 -> Connectors:SIL-2
- RR1, RR2, RR3, RR6, RR8: footprint connect:SIL-9 -> Connectors:SIL-9
- RR4, RR5, RR7: footprint discret:r_pack8 -> Discret:r_pack8
- W1, W2, W3: footprint connect:GS2 -> Connectors:GS2
- X1, X2: footprint discret:HC-18UV -> Discret:HC-18UV
- X3: value 4,433618MH -> 4.433618MHz; footprint discret:HC-18UH -> Discret:HC-18UH
Connections:
- net /ESVIDEO-RVB/BLANK- renamed /BLANK-
- net /ESVIDEO-RVB/BLUE renamed /BLUE_OUT
- net /ESVIDEO-RVB/BLUE_IN renamed /BLUE_IN
- net /ESVIDEO-RVB/CLAMP renamed /CLAMP
- net /ESVIDEO-RVB/CSYNCIN- renamed /CSYNCIN-
- net /ESVIDEO-RVB/GREEN renamed /GREEN_OUT
- net /ESVIDEO-RVB/GREEN_IN renamed /GREEN_IN
- net /ESVIDEO-RVB/OE_PAL- renamed /OE_PAL-
- net /ESVIDEO-RVB/RDCAD- renamed /RDCAD-
- net /ESVIDEO-RVB/RDCDA- renamed /RDCDA-
- net /ESVIDEO-RVB/RED_IN renamed /RED_IN
- net /ESVIDEO-RVB/WRCAD- renamed /WRCAD-
- net /ESVIDEO-RVB/WRCDA- renamed /WRCDA-
- net /RAMS/CAS0- renamed /CAS0-
- net /RAMS/CAS1- renamed /CAS1-
- net /RAMS/CAS2- renamed /CAS2-
- net /RAMS/CAS3- renamed /CAS3-
- net /RAMS/RAS0- renamed /RAS0-
- net /RAMS/RAS1- renamed /RAS1-
- net /RAMS/RAS2- renamed /RAS2-
- net /RAMS/RAS3- renamed /RAS3-
- net /RAMS/RAS4- renamed /RAS4-
- net /RAMS/RAS5- renamed /RAS5-
- net /RAMS/RAS6- renamed /RAS6-
- net /RAMS/RAS7- renamed /RAS7-
- net /RAMS/WRAM- renamed /WRAM-
- net /buspci.sch/BPCLK renamed /BPCLK
- net /buspci.sch/IRQ- renamed /IRQ-
- net /buspci.sch/PTADR- renamed /PTADR-
- net /buspci.sch/PTATN- renamed /PTATN-
- net /buspci.sch/PTBURST- renamed /PTBURST
- net /buspci.sch/PTNUM0 renamed /PTNUM0
- net /buspci.sch/PTNUM1 renamed /PTNUM1
- net /buspci.sch/PTRDY- renamed /PTRDY-
- net /buspci.sch/PTWR renamed /PTWR
- net /buspci.sch/RD- renamed //PCRD
- net /buspci.sch/RDEMPTY renamed /RDEMPTY
- net /buspci.sch/RDFIFO- renamed /RDFIFO-
- net /buspci.sch/SELECT- renamed /SELECT-
- net /buspci.sch/WR- renamed //PCWR
- net /buspci.sch/WRFIFO- renamed /WRFIFDO-
- net /buspci.sch/WRFULL renamed /WRFULL
- net /buspci.sch/X_IRQ renamed /X_IRQ
- net /graphic/ACCES_RAM- renamed /ACCES_RAM-
- net /graphic/ACQ_ON renamed /ACQ_ON
- net /graphic/BT812_RD- renamed /BT812_RD-
- net /graphic/BT812_WR- renamed /BT812_WR-
- net /graphic/CADCLK renamed /CLKCAD
- net /graphic/CDACLK renamed /CLKCDA
- net /graphic/CSYNC-OUT renamed /CSYNC-OUT
- net /graphic/F_PALIN renamed /F_PALIN
- net /graphic/HD_PAL- renamed /HD_PAL-
- net /graphic/IRQ_SLR renamed /IRQ_SRL
- net /graphic/VD_PAL- renamed /VD_PAL-
- net /graphic/X_CLK renamed /X_CLK
- net /graphic/X_DONE renamed /X_DONE
- net /graphic/X_PROG- renamed /X_PROG-
- net /modul/BLEU renamed /RED_OUT
- net /modul/COUT renamed /C_OUT
- net /modul/YOUT renamed /Y_OUT
- net /muxdata/DATA_WR renamed /WRITE_RAM
- net /muxdata/X_DIN renamed /X_DATA
- net /pal-ntsc.sch/RESET- renamed /SYSRST-
- net VCC renamed +5V
- U10 pad 101: (no net) -> Net-(U10-Pad101)
- U10 pad 105: (no net) -> Net-(U10-Pad105)
- U10 pad 106: (no net) -> Net-(U10-Pad106)
- U10 pad 107: (no net) -> Net-(U10-Pad107)
- U10 pad 127: (no net) -> Net-(U10-Pad127)
- U10 pad 129: (no net) -> Net-(U10-Pad129)
- U10 pad 131: (no net) -> Net-(U10-Pad131)
- U10 pad 150: (no net) -> Net-(U10-Pad150)
- U10 pad 152: (no net) -> Net-(U10-Pad152)
- U10 pad 154: (no net) -> Net-(U10-Pad154)
- U10 pad 25: (no net) -> Net-(U10-Pad25)
- U10 pad 26: (no net) -> Net-(U10-Pad26)
- U10 pad 27: (no net) -> Net-(U10-Pad27)
- U10 pad 28: (no net) -> Net-(U10-Pad28)
- U10 pad 29: (no net) -> Net-(U10-Pad29)
- U10 pad 32: (no net) -> Net-(U10-Pad32)
- U10 pad 33: (no net) -> Net-(U10-Pad33)
- U10 pad 35: (no net) -> Net-(U10-Pad35)
- U10 pad 37: (no net) -> Net-(U10-Pad37)
- U10 pad 38: (no net) -> Net-(U10-Pad38)
- U12 pad 67: (no net) -> Net-(U12-Pad67)
- U12 pad 68: (no net) -> Net-(U12-Pad68)
- U12 pad 69: (no net) -> Net-(U12-Pad69)
- U12 pad 70: (no net) -> Net-(U12-Pad70)
- U13 pad 67: (no net) -> Net-(U13-Pad67)
- U13 pad 68: (no net) -> Net-(U13-Pad68)
- U13 pad 69: (no net) -> Net-(U13-Pad69)
- U13 pad 70: (no net) -> Net-(U13-Pad70)
- U14 pad 67: (no net) -> Net-(U14-Pad67)
- U14 pad 68: (no net) -> Net-(U14-Pad68)
- U14 pad 69: (no net) -> Net-(U14-Pad69)
- U14 pad 70: (no net) -> Net-(U14-Pad70)
- U15 pad 67: (no net) -> Net-(U15-Pad67)
- U15 pad 68: (no net) -> Net-(U15-Pad68)
- U15 pad 69: (no net) -> Net-(U15-Pad69)
- U15 pad 70: (no net) -> Net-(U15-Pad70)
- U16 pad 67: (no net) -> Net-(U16-Pad67)
- U16 pad 68: (no net) -> Net-(U16-Pad68)
- U16 pad 69: (no net) -> Net-(U16-Pad69)
- U16 pad 70: (no net) -> Net-(U16-Pad70)
- U17 pad 67: (no net) -> Net-(U17-Pad67)
- U17 pad 68: (no net) -> Net-(U17-Pad68)
- U17 pad 69: (no net) -> Net-(U17-Pad69)
- U17 pad 70: (no net) -> Net-(U17-Pad70)
- U18 pad 67: (no net) -> Net-(U18-Pad67)
- U18 pad 68: (no net) -> Net-(U18-Pad68)
- U18 pad 69: (no net) -> Net-(U18-Pad69)
- U18 pad 70: (no net) -> Net-(U18-Pad70)
- U19 pad 67: (no net) -> Net-(U19-Pad67)
- U19 pad 68: (no net) -> Net-(U19-Pad68)
- U19 pad 69: (no net) -> Net-(U19-Pad69)
- U19 pad 70: (no net) -> Net-(U19-Pad70)
- U20 pad 1: (no net) -> Net-(U20-Pad1)
- U20 pad 3: (no net) -> Net-(U20-Pad3)
- U20 pad 4: (no net) -> Net-(U20-Pad4)
- U20 pad 5: (no net) -> Net-(U20-Pad5)
- U21 pad 6: (no net) -> Net-(U21-Pad6)
- U22 pad 10: (no net) -> Net-(U22-Pad10)
- U22 pad 14: (no net) -> Net-(U22-Pad14)
- U22 pad 15: (no net) -> Net-(U22-Pad15)
- U22 pad 16: (no net) -> Net-(U22-Pad16)
- U22 pad 27: (no net) -> Net-(U22-Pad27)
- U22 pad 3: (no net) -> Net-(U22-Pad3)
- U22 pad 30: (no net) -> Net-(U22-Pad30)
- U22 pad 4: (no net) -> Net-(U22-Pad4)
- U22 pad 5: (no net) -> Net-(U22-Pad5)
- U22 pad 6: (no net) -> Net-(U22-Pad6)
- U22 pad 65: (no net) -> Net-(U22-Pad65)
- U22 pad 66: (no net) -> Net-(U22-Pad66)
- U22 pad 73: (no net) -> Net-(U22-Pad73)
- U22 pad 76: (no net) -> Net-(U22-Pad76)
- U23 pad 100: (no net) -> Net-(U23-Pad100)
- U23 pad 2: (no net) -> Net-(U23-Pad2)
- U23 pad 31: (no net) -> Net-(U23-Pad31)
- U23 pad 33: (no net) -> Net-(U23-Pad33)
- U23 pad 49: (no net) -> Net-(U23-Pad49)
- U23 pad 50: (no net) -> Net-(U23-Pad50)
- U23 pad 58: (no net) -> Net-(U23-Pad58)
- U23 pad 60: (no net) -> Net-(U23-Pad60)
- U23 pad 62: (no net) -> Net-(U23-Pad62)
- U23 pad 68: (no net) -> Net-(U23-Pad68)
- U23 pad 76: (no net) -> Net-(U23-Pad76)
- U23 pad 79: (no net) -> Net-(U23-Pad79)
- U23 pad 98: (no net) -> Net-(U23-Pad98)
- U23 pad 99: (no net) -> Net-(U23-Pad99)
- U24 pad 121: (no net) -> Net-(U24-Pad121)
- U24 pad 84: (no net) -> Net-(U24-Pad84)
- U7 pad 8: (no net) -> Net-(U7-Pad8)
- U8 pad 4: (no net) -> Net-(U8-Pad4)
- U8 pad 5: (no net) -> Net-(U8-Pad5)
- U8 pad 74: (no net) -> Net-(U8-Pad74)
- U8 pad 77: (no net) -> Net-(U8-Pad77)
- U8 pad 81: (no net) -> Net-(U8-Pad81)
- U9 pad 27: (no net) -> Net-(U9-Pad27)
- U9 pad 30: (no net) -> Net-(U9-Pad30)
- U9 pad 5: (no net) -> Net-(U9-Pad5)
- U9 pad 6: (no net) -> Net-(U9-Pad6)
