File: demos/electric/electric.sch (KiCad schematic (older format))
At the start: 97 parts

Commit message: Update demo files
Parts:
- EC11, EC12, EC13, EC14, EC15, EC16, EC17, EC18, EC19, EC31, EC41, EC42, EC43, EC44: value C_3X1.5MM2 -> C_3x1.5mm2; symbol C_3X1.5MM2 -> C_3x1.5mm2
- EC20, EC21, EC22, EC23, EC24, EC25, EC26, EC28, EC29, EC30, EC32, EC33, EC34, EC35, EC36, EC37, EC38, EC39, EC? (x2): value C_3X2.5MM2 -> C_3x2.5mm2; symbol C_3X2.5MM2 -> C_3x2.5mm2
- EC27: value C_3X6MM2 -> C_3x6mm2; symbol C_3X6MM2 -> C_3x6mm2
- EG1: value G_TH_3KVA -> G_Th_3KVA; symbol G_TH_3KVA -> G_Th_3KVA; Champ4 (none) -> automatique; Champ5 (none) -> diesel
- EJ1, EJ2, EJ3, EJ4: value J_40A_30MA -> J_40A_30mA; symbol J_40A_30MA -> J_40A_30mA
- EO1: Champ4 (none) -> rallongée
- ER01, ER02: value R_16A_30MA -> R_16A_30mA; symbol R_16A_30MA -> R_16A_30mA
Other:
- note added: "Servitudes\npermanentes\nprimaires"
- note added: "Servitudes\npermanentes\nsecondaires"
- note removed: "Servitudes"
- note removed: "permanentes"
- note removed: "primaires"
- note removed: "secondaires"

Commit message: 3D viewer: speed up the silkscreen layer generation (not perfect, but it help).
Parts:
- EV2: symbol V_F50HZ -> V_F50Hz
Connections:
- wire segments 135 -> 82
Changed lines of the file:
@@
 EESchema Schematic File Version 2
+LIBS:electric-rescue
 LIBS:power
 LIBS:elec-unifil
@@
 LIBS:regul
 LIBS:electric-cache
-EELAYER 24 0
+EELAYER 25 0
 EELAYER END
 $Descr A4 11693 8268
@@
 Connection ~ 8250 2900
 Wire Wire Line
-	8250 2400 8350 2400
-Wire Wire Line
-	8150 2900 8250 2900
-Wire Wire Line
-	8250 2900 8350 2900
+	5250 2400 8350 2400
+Wire Wire Line
+	5250 2900 8350 2900
 Wire Wire Line
 	4450 2400 4850 2400
 Wire Wire Line
-	4850 1900 4550 1900
-Wire Wire Line
-	4550 1900 4450 1900
-Wire Wire Line
-	5600 1900 5700 1900
+	4450 1900 4850 1900
+Wire Wire Line
+	5250 1900 5700 1900
 Wire Notes Line
 	5500 550  5600 550
@@
 	5500 1650 5500 550
 Wire Notes Line
-	5550 1650 5500 1650
-Wire Notes Line
-	5500 2200 5550 2200
+	5500 1650 8100 1650
+Wire Notes Line
+	5500 2200 8100 2200
 Wire Notes Line
 	5500 1700 5500 2200
 Wire Notes Line
-	5550 1700 5500 1700
-Wire Wire Line
-	5250 1900 5600 1900
+	5500 1700 8100 1700
 Connection ~ 3950 1900
 Connection ~ 3150 2450
 Connection ~ 4550 1900
 Wire Wire Line
-	2600 800  2600 1400
-Wire Wire Line
-	4550 800  2600 800
+	2600 800  2600 1900
+Wire Wire Line
+	2600 800  5700 800
 Wire Wire Line
 	4550 800  4550 1900
 Wire Wire Line
-	4950 800  4550 800
-Wire Wire Line
-	5350 2900 5250 2900
-Wire Wire Line
-	5350 2400 5250 2400
-Wire Wire Line
-	4850 2900 4850 2400
+	4850 2400 4850 2900
 Wire Wire Line
 	3750 2450 4050 2450
@@
 	3950 1900 3950 2400
 Wire Wire Line
-	3850 1950 4050 1950
-Wire Wire Line
-	3850 1900 3950 1900
-Wire Wire Line
-	3950 1900 4050 1900
-Wire Wire Line
-	3150 2450 3350 2450
-Wire Wire Line
-	3150 1950 3200 1950
+	3150 1950 4050 1950
+Wire Wire Line
+	3100 1900 4050 1900
+Wire Wire Line
+	3000 2450 3350 2450
 Wire Wire Line
 	3150 2450 3150 1950
 Wire Wire Line
-	3000 2450 3150 2450
-Wire Wire Line
-	3100 1900 3150 1900
-Wire Wire Line
 	3100 2400 3100 1900
 Wire Wire Line
@@
 	3850 2050 3850 2850
 Wire Notes Line
-	3800 2050 3850 2050
-Wire Notes Line
-	3750 2050 3800 2050
+	3250 2050 3850 2050
 Wire Notes Line
 	3250 2050 3250 3100
 Wire Notes Line
-	4700 1150 4700 2850
-Wire Notes Line
-	4750 1150 4700 1150
-Wire Notes Line
-	5400 3100 5350 3100
+	4700 2850 4700 1150
+Wire Notes Line
+	4700 1150 5400 1150
 Wire Notes Line
 	5400 1150 5400 3100
-Wire Notes Line
-	5350 1150 5400 1150
 Wire Notes Line
 	8100 6000 8100 3150
@@
 Text Notes 4150 3000 0    60   ~ 0
 AGBT
-Wire Notes Line
-	5350 1150 4750 1150
-Wire Notes Line
-	3250 2050 3750 2050
-Wire Wire Line
-	3850 1950 3200 1950
-Wire Wire Line
-	3150 1900 3850 1900
-Wire Wire Line
-	2600 1900 2600 1400
 Wire Wire Line
 	1550 950  1800 950
@@
 	1700 2150 1750 2150
 Wire Wire Line
-	1950 3350 1700 3350
-Wire Wire Line
-	1950 3850 1700 3850
-Wire Wire Line
-	1950 4350 1700 4350
-Wire Wire Line
-	1950 4850 1700 4850
+	1700 3350 5700 3350
+Wire Wire Line
+	1700 3850 5400 3850
+Wire Wire Line
+	1700 4350 2350 4350
+Wire Wire Line
+	1700 4850 2050 4850
 Wire Wire Line
 	850  4850 1200 4850
@@
 Connection ~ 2050 6600
 Wire Wire Line
-	2050 4850 1950 4850
-Wire Wire Line
-	2050 6600 2050 4850
-Wire Wire Line
-	2050 7550 2050 7300
-Wire Wire Line
-	2050 7300 2050 6950
-Wire Wire Line
-	2050 6950 2050 6600
-Wire Wire Line
-	2350 7550 2050 7550
+	2050 4850 2050 7550
+Wire Wire Line
+	2050 7550 2350 7550
 Wire Wire Line
 	2350 7300 2050 7300
@@
 	2150 4100 2150 6300
 Wire Wire Line
-	5400 6100 5450 6100
+	5400 6100 8350 6100
 Wire Wire Line
 	5400 3850 5400 6100
-Wire Wire Line
-	1950 3850 5400 3850
 Wire Notes Line
 	5500 6000 8100 6000
@@
 	8150 4200 11100 4200
 Wire Wire Line
-	8250 4450 8250 4800
-Wire Wire Line
-	8250 4800 8250 5400
-Wire Wire Line
-	8250 5400 8250 5750
-Wire Wire Line
-	8250 5750 8250 6100
+	8250 4450 8250 6100
 Wire Wire Line
 	8750 5100 8750 5400
@@
 	8150 2650 11100 2650
 Wire Notes Line
-	11100 2600 11100 2200
+	11100 500  11100 2600
 Wire Notes Line
 	8150 2600 11100 2600
 Wire Notes Line
-	8150 2200 8150 2600
-Wire Notes Line
-	5600 2200 5550 2200
-Wire Notes Line
-	8100 2200 5600 2200
+	8150 500  8150 2600
 Wire Notes Line
 	8100 1700 8100 2200
 Wire Notes Line
-	5550 1700 8100 1700
-Wire Notes Line
 	8100 1650 8100 550
 Wire Notes Line
-	5550 1650 8100 1650
-Wire Notes Line
 	8100 550  5550 550
 Wire Notes Line
 	11100 500  8150 500
 Wire Notes Line
-	11100 2200 11100 500
-Wire Notes Line
 	11050 500  11050 500
-Wire Notes Line
-	8150 500  8150 2200
 $Comp
 L D_06A ED30
@@
 	8250 3950 8350 3950
 Wire Wire Line
-	8250 3250 8250 3600
-Wire Wire Line
-	8250 3600 8250 3950
+	8250 2900 8250 3950
 Wire Wire Line
 	8350 3250 8250 3250
 Wire Wire Line
-	8250 2900 8250 3250
-Wire Wire Line
-	5350 2900 8150 2900
-Wire Wire Line
-	8250 650  8250 1000
-Wire Wire Line
-	8250 1000 8250 1350
-Wire Wire Line
-	8250 1350 8250 1700
-Wire Wire Line
-	8250 1700 8250 2050
-Wire Wire Line
-	8250 2050 8250 2400
+	8250 650  8250 2400
 Text HLabel 6500 800  2    60   Output ~ 0
 EC12
@@
 $EndComp
 Connection ~ 850  2750
-Wire Wire Line
-	5450 6100 8250 6100
-Wire Wire Line
-	8250 6100 8350 6100
 Connection ~ 8250 6100
 Connection ~ 8250 4800
@@
 Wire Wire Line
 	8350 4450 8250 4450
-Wire Wire Line
-	5350 2400 8250 2400
-Wire Wire Line
-	2350 4350 2250 4350
-Wire Wire Line
-	2250 4350 1950 4350
 Connection ~ 2250 4350
 Connection ~ 2250 5750
@@
 	2350 4700 2250 4700
 Wire Wire Line
-	2350 5050 2250 5050
-Wire Wire Line
-	2350 5400 2250 5400
-Wire Wire Line
-	2350 5750 2250 5750
+	2250 5050 2350 5050
+Wire Wire Line
+	2250 5400 2350 5400
+Wire Wire Line
+	2250 5750 2350 5750
 Wire Wire Line
 	2250 6100 2350 6100
 Wire Wire Line
-	2250 4350 2250 4700
-Wire Wire Line
-	2250 4700 2250 5050
-Wire Wire Line
-	2250 5050 2250 5400
-Wire Wire Line
-	2250 5400 2250 5750
-Wire Wire Line
-	2250 5750 2250 6100
+	2250 4350 2250 6100
 $Comp
 L D_10A ED73
@@
 Connection ~ 5600 3350
 Wire Wire Line
-	5700 3350 5600 3350
-Wire Wire Line
-	5600 3350 1950 3350
-Wire Wire Line
-	5700 5450 5600 5450
-Wire Wire Line
-	5700 5100 5600 5100
-Wire Wire Line
-	5700 4750 5600 4750
-Wire Wire Line
-	5700 4400 5600 4400
-Wire Wire Line
-	5700 4050 5600 4050
+	5600 5450 5700 5450
+Wire Wire Line
+	5600 5100 5700 5100
+Wire Wire Line
+	5600 4750 5700 4750
+Wire Wire Line
+	5600 4400 5700 4400
+Wire Wire Line
+	5600 4050 5700 4050
 Wire Wire Line
 	5700 3700 5600 3700
@@
 	5600 5800 5700 5800
 Wire Wire Line
-	5600 3350 5600 3700
-Wire Wire Line
-	5600 3700 5600 4050
-Wire Wire Line
-	5600 4050 5600 4400
-Wire Wire Line
-	5600 4400 5600 4750
-Wire Wire Line
-	5600 4750 5600 5100
-Wire Wire Line
-	5600 5100 5600 5450
-Wire Wire Line
-	5600 5450 5600 5800
+	5600 3350 5600 5800
 $Comp
 L D_10A ED47
@@
 Connection ~ 8250 1350
 Connection ~ 8250 1000
-Connection ~ 8250 1000
-Connection ~ 8250 1000
 Wire Wire Line
 	8250 1000 8350 1000
@@
 	5600 1150 5700 1150
 Wire Wire Line
-	4950 800  5600 800
-Wire Wire Line
-	5600 800  5700 800
-Wire Wire Line
-	5600 1500 5600 1150
-Wire Wire Line
-	5600 1150 5600 800
-Wire Wire Line
-	5700 1500 5600 1500
+	5600 800  5600 1500
+Wire Wire Line
+	5600 1500 5700 1500
 $Comp
 L D_06A ED15
@@
 Connection ~ 850  3350
 Wire Wire Line
-	850  1350 850  1500
-Wire Wire Line
-	850  1500 850  2750
-Wire Wire Line
-	850  2750 850  3350
-Wire Wire Line
-	850  3350 850  3850
-Wire Wire Line
-	850  3850 850  4350
-Wire Wire Line
-	850  4350 850  4850
-Connection ~ 850  1500
+	850  1350 850  4850
 $Comp
 L O_600VA EO2
@@
 Connection ~ 4350 1900
 $Comp
-L V_F50HZ EV2
+L V_F50Hz EV2
 U 1 1 4162DD75
 P 2400 1400

Commit message: merge from production git:30df041
Parts:
- gave numbers to parts that had none: 2
- renumbered EQ1a to EQ1a101, EQ1b to EQ1b101, ER01 to ER1, ER02 to ER2, EW01 to EW1
Other:
- moved on the sheet: ED13, ED14, ED60, ED64
Changed lines of the file:
@@
 EESchema Schematic File Version 2
-LIBS:electric-rescue
 LIBS:power
 LIBS:elec-unifil
 LIBS:device
 LIBS:conn
-LIBS:regul
 LIBS:electric-cache
-EELAYER 25 0
+EELAYER 26 0
 EELAYER END
 $Descr A4 11693 8268
@@
 	850  3350 1200 3350
 $Comp
-L R_16A_30mA ER01
+L R_16A_30mA ER1
 U 1 1 416242BF
 P 1450 2150
-F 0 "ER01" H 1400 2380 40  0000 C CNN
+F 0 "ER1" H 1400 2380 40  0000 C CNN
 F 1 "R_16A_30mA" H 1450 1950 40  0000 C CNN
 F 2 "Courbe D" H 1450 1900 30  0000 C CNN
@@
 	850  2750 1200 2750
 $Comp
-L C_3x2.5mm2 EC?
+L C_3x2.5mm2 EC102
 U 1 1 41652EC2
 P 2950 6950
-F 0 "EC?" H 2780 7080 40  0000 C CNN
+F 0 "EC102" H 2780 7080 40  0000 C CNN
 F 1 "C_3x2.5mm2" H 2950 6850 40  0000 C CNN
 F 2 "" H 2950 6950 60  0001 C CNN
@@
 $EndComp
 $Comp
-L C_3x2.5mm2 EC?
+L C_3x2.5mm2 EC101
 U 1 1 41642129
 P 2950 6600
-F 0 "EC?" H 2780 6730 40  0000 C CNN
+F 0 "EC101" H 2780 6730 40  0000 C CNN
 F 1 "C_3x2.5mm2" H 2950 6500 40  0000 C CNN
 F 2 "" H 2950 6600 60  0001 C CNN
@@
 $Comp
 L D_16A ED54
-U 1 1 4162F875
+U 1 1 5831E95C
 P 2550 5750
 F 0 "ED54" H 2390 5870 40  0000 C CNN
@@
 $Comp
 L D_16A ED50
-U 1 1 4162F848
+U 1 1 5831E958
 P 2550 4350
 F 0 "ED50" H 2390 4470 40  0000 C CNN
@@
 $Comp
 L D_16A ED63
-U 1 1 4162F862
+U 1 1 5831E95B
 P 8550 5750
 F 0 "ED63" H 8390 5870 40  0000 C CNN
@@
 $Comp
 L D_16A ED62
-U 1 1 4162F856
+U 1 1 5831E95A
 P 8550 5400
 F 0 "ED62" H 8390 5520 40  0000 C CNN
@@
 $Comp
 L D_16A ED61
-U 1 1 4162F84D
+U 1 1 5831E959
 P 8550 4800
 F 0 "ED61" H 8390 4920 40  0000 C CNN
@@
 $Comp
 L D_06A ED32
-U 1 1 4162F2EE
+U 1 1 5831E955
 P 8550 3600
 F 0 "ED32" H 8390 3720 40  0000 C CNN
@@
 $Comp
 L D_06A ED33
-U 1 1 4162F2D8
+U 1 1 5831E954
 P 8550 3950
 F 0 "ED33" H 8390 4070 40  0000 C CNN
@@
 $Comp
 L D_06A ED31
-U 1 1 4162F2D8
+U 1 1 5831E953
 P 8550 3250
 F 0 "ED31" H 8390 3370 40  0000 C CNN
@@
 $Comp
 L D_06A ED11
-U 1 1 4162F301
+U 1 1 5831E957
 P 8550 650
 F 0 "ED11" H 8390 770 40  0000 C CNN
@@
 $Comp
 L D_06A ED12
-U 1 1 4162F2F6
+U 1 1 5831E956
 P 8550 1000
 F 0 "ED12" H 8390 1120 40  0000 C CNN
@@
 $Comp
 L D_10A ED25
-U 1 1 4162F22A
+U 1 1 5831E952
 P 5900 1900
 F 0 "ED25" H 5740 2020 40  0000 C CNN
@@
 $Comp
 L D_10A ED22
-U 1 1 4162F1F7
+U 1 1 5831E951
 P 5900 1500
 F 0 "ED22" H 5740 1620 40  0000 C CNN
@@
 $Comp
 L D_10A ED21
-U 1 1 4162F1F0
+U 1 1 5831E950
 P 5900 1150
 F 0 "ED21" H 5750 1250 40  0000 C CNN
@@
 $Comp
 L D_10A ED20
-U 1 1 4162F1CA
+U 1 1 5831E94F
 P 5900 800
 F 0 "ED20" H 5740 920 40  0000 C CNN
@@
 $EndComp
 $Comp
-L Q_25A_2F2O EQ1b
+L Q_25A_2F2O EQ1b101
 U 1 1 416245A7
 P 2800 2400
-F 0 "EQ1b" H 2700 2550 40  0000 C CNN
+F 0 "EQ1b101" H 2700 2550 40  0000 C CNN
 F 1 "Q_25A_2F2O" H 2800 2260 40  0000 C CNN
 F 2 "" H 2800 2400 60  0001 C CNN
@@
 $EndComp
 $Comp
-L Q_25A_2F2O EQ1a
+L Q_25A_2F2O EQ1a101
 U 1 1 41624555
 P 2000 2400
-F 0 "EQ1a" H 1900 2550 40  0000 C CNN
+F 0 "EQ1a101" H 1900 2550 40  0000 C CNN
 F 1 "Q_25A_2F2O" H 2000 2260 40  0000 C CNN
 F 2 "" H 2000 2400 60  0001 C CNN
@@
 $EndComp
 $Comp
-L R_16A_30mA ER02
+L R_16A_30mA ER2
 U 1 1 416242F0
 P 1450 2750
-F 0 "ER02" H 1240 2930 40  0000 C CNN
+F 0 "ER2" H 1240 2930 40  0000 C CNN
 F 1 "R_16A_30mA" H 1450 2550 40  0000 C CNN
 F 2 "Courbe B" H 1450 2500 30  0000 C CNN
@@
 	1350 1350 1350 1500
 $Comp
-L W_15KA EW01
+L W_15KA EW1
 U 1 1 41618802
 P 1800 1150
-F 0 "EW01" H 1800 1300 40  0000 C CNN
+F 0 "EW1" H 1800 1300 40  0000 C CNN
 F 1 "W_15KA" H 1800 950 40  0000 C CNN
 F 2 "" H 1800 1150 60  0001 C CNN
