File: demos/complex_hierarchy/ampli_ht.sch (KiCad schematic (older format))
At the start: 29 parts, among them P5 CONN_2, P6 CONN_2, Q5 MPAS92, Q6 MPAS42, Q7 MPAS92, Q8 MPAS42, U4 LM358N

Commit message: Demos: make a private library for each demo, to avoid issues when using modified kicad new schematic libraries
Connections:
- wire segments 80 -> 67
Changed lines of the file:
@@
 EESchema Schematic File Version 2
+LIBS:complex_hierarchy_schlib
 LIBS:power
-LIBS:device
-LIBS:transistors
-LIBS:conn
-LIBS:linear
-LIBS:regul
-LIBS:interface
-LIBS:special
 LIBS:complex_hierarchy-cache
 EELAYER 25 0
@@
 	9800 4450 9700 4450
 Wire Wire Line
-	9800 4150 9800 4300
-Wire Wire Line
-	9800 4300 9800 4450
+	9800 4150 9800 4450
 Wire Wire Line
 	9800 4150 9700 4150
@@
 	6900 5400 7150 5400
 Wire Wire Line
-	2700 2000 2850 2000
-Wire Wire Line
-	2850 2000 3000 2000
+	2700 2000 3000 2000
 Connection ~ 7300 3300
 Wire Wire Line
-	7300 3200 7300 3300
-Wire Wire Line
-	7300 3300 7300 3350
+	7300 3200 7300 3350
 Wire Wire Line
 	5400 6400 5600 6400
@@
 Connection ~ 5450 2400
 Wire Wire Line
-	5450 3000 5450 2400
-Wire Wire Line
-	5450 2400 5450 1600
+	5450 3000 5450 1600
 Wire Wire Line
 	5450 1600 4550 1600
 Wire Wire Line
-	3500 2000 3600 2000
-Wire Wire Line
-	3600 2000 3700 2000
+	3500 2000 3700 2000
 Wire Wire Line
 	7000 5100 7000 5200
@@
 	5850 5500 5900 5500
 Wire Wire Line
-	4350 3000 5150 3000
-Wire Wire Line
-	5150 3000 5450 3000
+	4350 3000 5450 3000
 Wire Wire Line
 	4350 2000 4200 2000
@@
 Connection ~ 8100 4800
 Wire Wire Line
-	7900 3500 7900 3700
-Wire Wire Line
-	7900 3700 7900 3800
-Wire Wire Line
-	7900 4700 7900 4800
-Wire Wire Line
-	7900 4800 7900 4900
+	7900 3500 7900 3800
+Wire Wire Line
+	7900 4700 7900 4900
 Wire Wire Line
 	9800 4300 10400 4300
@@
 Connection ~ 8900 4450
 Wire Wire Line
-	8900 5350 8900 5400
-Wire Wire Line
-	8900 5400 8900 6400
+	8900 5350 8900 6400
 Connection ~ 8900 5400
 $Comp
@@
 $EndComp
 $Comp
-L GND #PWR020
+L GND #PWR019
 U 1 1 4B6168A3
 P 8100 6000
-AR Path="/4B3A13A4/4B6168A3" Ref="#PWR020"  Part="1"
-AR Path="/4B3A1333/4B6168A3" Ref="#PWR036"  Part="1"
-F 0 "#PWR020" H 8100 6000 30  0001 C CNN
+AR Path="/4B3A13A4/4B6168A3" Ref="#PWR019"  Part="1"
+AR Path="/4B3A1333/4B6168A3" Ref="#PWR035"  Part="1"
+F 0 "#PWR035" H 8100 6000 30  0001 C CNN
 F 1 "GND" H 8100 5930 30  0001 C CNN
 F 2 "" H 8100 6000 60  0001 C CNN
@@
 $EndComp
 $Comp
-L GND #PWR037
+L GND #PWR036
 U 1 1 4B4F364A
 P 2850 2550
-AR Path="/4B3A1333/4B4F364A" Ref="#PWR037"  Part="1"
-AR Path="/4B3A13A4/4B4F364A" Ref="#PWR021"  Part="1"
-F 0 "#PWR021" H 2850 2550 30  0001 C CNN
+AR Path="/4B3A1333/4B4F364A" Ref="#PWR036"  Part="1"
+AR Path="/4B3A13A4/4B4F364A" Ref="#PWR020"  Part="1"
+F 0 "#PWR036" H 2850 2550 30  0001 C CNN
 F 1 "GND" H 2850 2480 30  0001 C CNN
 F 2 "" H 2850 2550 60  0001 C CNN
@@
 $EndComp
 $Comp
-L -VAA #PWR022
+L -VAA #PWR021
 U 1 1 4B4B1086
 P 6300 5850
-AR Path="/4B3A13A4/4B4B1086" Ref="#PWR022"  Part="1"
-AR Path="/4B3A1333/4B4B1086" Ref="#PWR038"  Part="1"
-F 0 "#PWR022" H 6300 5950 20  0001 C CNN
+AR Path="/4B3A13A4/4B4B1086" Ref="#PWR021"  Part="1"
+AR Path="/4B3A1333/4B4B1086" Ref="#PWR037"  Part="1"
+F 0 "#PWR037" H 6300 5950 20  0001 C CNN
 F 1 "-VAA" H 6300 5950 40  0000 C CNN
 F 2 "" H 6300 5850 60  0001 C CNN
@@
 $EndComp
 $Comp
-L -VAA #PWR023
+L -VAA #PWR022
 U 1 1 4B4B1080
 P 4750 2850
-AR Path="/4B3A13A4/4B4B1080" Ref="#PWR023"  Part="1"
-AR Path="/4B3A1333/4B4B1080" Ref="#PWR039"  Part="1"
-F 0 "#PWR023" H 4750 2950 20  0001 C CNN
+AR Path="/4B3A13A4/4B4B1080" Ref="#PWR022"  Part="1"
+AR Path="/4B3A1333/4B4B1080" Ref="#PWR038"  Part="1"
+F 0 "#PWR038" H 4750 2950 20  0001 C CNN
 F 1 "-VAA" H 4750 2950 40  0000 C CNN
 F 2 "" H 4750 2850 60  0001 C CNN
@@
 $EndComp
 $Comp
-L GND #PWR024
+L GND #PWR023
 U 1 1 4B3A137A
 P 8600 5300
-AR Path="/4B3A13A4/4B3A137A" Ref="#PWR024"  Part="1"
-AR Path="/4B3A1333/4B3A137A" Ref="#PWR040"  Part="1"
-F 0 "#PWR024" H 8600 5300 30  0001 C CNN
+AR Path="/4B3A13A4/4B3A137A" Ref="#PWR023"  Part="1"
+AR Path="/4B3A1333/4B3A137A" Ref="#PWR039"  Part="1"
+F 0 "#PWR039" H 8600 5300 30  0001 C CNN
 F 1 "GND" H 8600 5230 30  0001 C CNN
 F 2 "" H 8600 5300 60  0001 C CNN
@@
 $EndComp
 $Comp
-L GND #PWR025
+L GND #PWR024
 U 1 1 4B3A1378
 P 7000 5200
-AR Path="/4B3A13A4/4B3A1378" Ref="#PWR025"  Part="1"
-AR Path="/4B3A1333/4B3A1378" Ref="#PWR041"  Part="1"
-F 0 "#PWR025" H 7000 5200 30  0001 C CNN
+AR Path="/4B3A13A4/4B3A1378" Ref="#PWR024"  Part="1"
+AR Path="/4B3A1333/4B3A1378" Ref="#PWR040"  Part="1"
+F 0 "#PWR040" H 7000 5200 30  0001 C CNN
 F 1 "GND" H 7000 5130 30  0001 C CNN
 F 2 "" H 7000 5200 60  0001 C CNN
@@
 $EndComp
 $Comp
-L GND #PWR026
+L GND #PWR025
 U 1 1 4B3A1373
 P 7300 3950
-AR Path="/4B3A13A4/4B3A1373" Ref="#PWR026"  Part="1"
-AR Path="/4B3A1333/4B3A1373" Ref="#PWR042"  Part="1"
-F 0 "#PWR026" H 7300 3950 30  0001 C CNN
+AR Path="/4B3A13A4/4B3A1373" Ref="#PWR025"  Part="1"
+AR Path="/4B3A1333/4B3A1373" Ref="#PWR041"  Part="1"
+F 0 "#PWR041" H 7300 3950 30  0001 C CNN
 F 1 "GND" H 7300 3880 30  0001 C CNN
 F 2 "" H 7300 3950 60  0001 C CNN
@@
 $EndComp
 $Comp
-L +12V #U027
+L +12V #U026
 U 1 1 4B3A136F
 P 6300 4950
-AR Path="/4B3A13A4/4B3A136F" Ref="#U027"  Part="1"
-AR Path="/4B3A1333/4B3A136F" Ref="#U043"  Part="1"
-F 0 "#U027" H 6300 4900 20  0001 C CNN
+AR Path="/4B3A13A4/4B3A136F" Ref="#U026"  Part="1"
+AR Path="/4B3A1333/4B3A136F" Ref="#U042"  Part="1"
+F 0 "#U042" H 6300 4900 20  0001 C CNN
 F 1 "+12V" H 6300 5050 40  0000 C CNN
 F 2 "" H 6300 4950 60  0001 C CNN
@@
 $EndComp
 $Comp
-L GND #PWR028
+L GND #PWR027
 U 1 1 4B3A136A
 P 1800 2250
-AR Path="/4B3A13A4/4B3A136A" Ref="#PWR028"  Part="1"
-AR Path="/4B3A1333/4B3A136A" Ref="#PWR044"  Part="1"
-F 0 "#PWR028" H 1800 2250 30  0001 C CNN
+AR Path="/4B3A13A4/4B3A136A" Ref="#PWR027"  Part="1"
+AR Path="/4B3A1333/4B3A136A" Ref="#PWR043"  Part="1"
+F 0 "#PWR043" H 1800 2250 30  0001 C CNN
 F 1 "GND" H 1800 2180 30  0001 C CNN
 F 2 "" H 1800 2250 60  0001 C CNN
@@
 $EndComp
 $Comp
-L GND #PWR029
+L GND #PWR028
 U 1 1 4B3A1369
 P 4000 2850
-AR Path="/4B3A13A4/4B3A1369" Ref="#PWR029"  Part="1"
-AR Path="/4B3A1333/4B3A1369" Ref="#PWR045"  Part="1"
-F 0 "#PWR029" H 4000 2850 30  0001 C CNN
+AR Path="/4B3A13A4/4B3A1369" Ref="#PWR028"  Part="1"
+AR Path="/4B3A1333/4B3A1369" Ref="#PWR044"  Part="1"
+F 0 "#PWR044" H 4000 2850 30  0001 C CNN
 F 1 "GND" H 4000 2780 30  0001 C CNN
 F 2 "" H 4000 2850 60  0001 C CNN
@@
 $EndComp
 $Comp
-L GND #PWR030
+L GND #PWR029
 U 1 1 4B3A1363
 P 10250 4550
-AR Path="/4B3A13A4/4B3A1363" Ref="#PWR030"  Part="1"
-AR Path="/4B3A1333/4B3A1363" Ref="#PWR046"  Part="1"
-F 0 "#PWR030" H 10250 4550 30  0001 C CNN
+AR Path="/4B3A13A4/4B3A1363" Ref="#PWR029"  Part="1"
+AR Path="/4B3A1333/4B3A1363" Ref="#PWR045"  Part="1"
+F 0 "#PWR045" H 10250 4550 30  0001 C CNN
 F 1 "GND" H 10250 4480 30  0001 C CNN
 F 2 "" H 10250 4550 60  0001 C CNN
@@
 $EndComp
 $Comp
-L GND #PWR031
+L GND #PWR030
 U 1 1 4B3A1361
 P 4850 6400
-AR Path="/4B3A13A4/4B3A1361" Ref="#PWR031"  Part="1"
-AR Path="/4B3A1333/4B3A1361" Ref="#PWR047"  Part="1"
-F 0 "#PWR031" H 4850 6400 30  0001 C CNN
+AR Path="/4B3A13A4/4B3A1361" Ref="#PWR030"  Part="1"
+AR Path="/4B3A1333/4B3A1361" Ref="#PWR046"  Part="1"
+F 0 "#PWR046" H 4850 6400 30  0001 C CNN
 F 1 "GND" H 4850 6330 30  0001 C CNN
 F 2 "" H 4850 6400 60  0001 C CNN
@@
 $EndComp
 $Comp
-L HT #PWR032
+L HT #PWR031
 U 1 1 4B3A135F
 P 7300 2250
-AR Path="/4B3A13A4/4B3A135F" Ref="#PWR032"  Part="1"
-AR Path="/4B3A1333/4B3A135F" Ref="#PWR048"  Part="1"
-F 0 "#PWR032" H 7300 2370 20  0001 C CNN
+AR Path="/4B3A13A4/4B3A135F" Ref="#PWR031"  Part="1"
+AR Path="/4B3A1333/4B3A135F" Ref="#PWR047"  Part="1"
+F 0 "#PWR047" H 7300 2370 20  0001 C CNN
 F 1 "HT" H 7300 2340 40  0000 C CNN
 F 2 "" H 7300 2250 60  0001 C CNN
@@
 $EndComp
 $Comp
-L HT #PWR033
+L HT #PWR032
 U 1 1 4B3A135E
 P 7900 2450
-AR Path="/4B3A13A4/4B3A135E" Ref="#PWR033"  Part="1"
-AR Path="/4B3A1333/4B3A135E" Ref="#PWR049"  Part="1"
-F 0 "#PWR033" H 7900 2570 20  0001 C CNN
+AR Path="/4B3A13A4/4B3A135E" Ref="#PWR032"  Part="1"
+AR Path="/4B3A1333/4B3A135E" Ref="#PWR048"  Part="1"
+F 0 "#PWR048" H 7900 2570 20  0001 C CNN
 F 1 "HT" H 7900 2540 40  0000 C CNN
 F 2 "" H 7900 2450 60  0001 C CNN
@@
 $EndComp
 $Comp
-L HT #PWR034
+L HT #PWR033
 U 1 1 4B3A135D
 P 8600 3300
-AR Path="/4B3A13A4/4B3A135D" Ref="#PWR034"  Part="1"
-AR Path="/4B3A1333/4B3A135D" Ref="#PWR050"  Part="1"
-F 0 "#PWR034" H 8600 3420 20  0001 C CNN
+AR Path="/4B3A13A4/4B3A135D" Ref="#PWR033"  Part="1"
+AR Path="/4B3A1333/4B3A135D" Ref="#PWR049"  Part="1"
+F 0 "#PWR049" H 8600 3420 20  0001 C CNN
 F 1 "HT" H 8600 3390 40  0000 C CNN
 F 2 "" H 8600 3300 60  0001 C CNN
@@
 $EndComp
 $Comp
-L +12V #U035
+L +12V #U034
 U 1 1 4B3A135B
 P 4750 1950
-AR Path="/4B3A13A4/4B3A135B" Ref="#U035"  Part="1"
-AR Path="/4B3A1333/4B3A135B" Ref="#U051"  Part="1"
-F 0 "#U035" H 4750 1900 20  0001 C CNN
+AR Path="/4B3A13A4/4B3A135B" Ref="#U034"  Part="1"
+AR Path="/4B3A1333/4B3A135B" Ref="#U050"  Part="1"
+F 0 "#U050" H 4750 1900 20  0001 C CNN
 F 1 "+12V" H 4750 2050 40  0000 C CNN
 F 2 "" H 4750 1950 60  0001 C CNN
@@
 	7900 4200 7900 4300
 Wire Wire Line
-	8600 4450 8900 4450
-Wire Wire Line
-	8900 4450 9200 4450
+	8600 4450 9200 4450
 Wire Wire Line
 	8600 4450 8600 4600
 Wire Wire Line
-	8600 4150 9100 4150
-Wire Wire Line
-	9100 4150 9200 4150
+	8600 4150 9200 4150
 Wire Wire Line
 	8600 4150 8600 3900
@@
 	2850 2550 2850 2500
 Wire Wire Line
-	4350 2000 4350 2200
-Wire Wire Line
-	4350 2200 4350 2300
+	4350 2000 4350 2300
 Wire Wire Line
 	4350 2200 4000 2200
@@
 	7900 2450 7900 2500
 Wire Wire Line
-	8300 4800 8100 4800
-Wire Wire Line
-	8100 4800 7900 4800
+	7900 4800 8300 4800
 Connection ~ 7900 4800
 Wire Wire Line

Commit message: Eeschema: BOM dialog: fix some minor issues when displaying messages. Cvpcb: fix Bug #1470201 (select next/previous unlinked comp and clear links not working well) demo/complex_hierarchy: use our new schematic symbols.
Parts:
- C12, C6, C7, C8: footprint (none) -> discret:C2
- D5, D6, D7, D8: footprint (none) -> discret:D3; symbol DIODE -> D_Small
- P5, P6: footprint (none) -> connect:bornier2
- Q5, Q6, Q7, Q8: footprint (none) -> discret:TO92-CBE
- R10, R13, R14, R15, R16, R17, R18, R19, R21, R22, R23, R25, R26: footprint (none) -> discret:R3-LARGE_PADS
- RV2: footprint (none) -> discret:RV2
- U4: footprint (none) -> dip_sockets:DIP-8__300_ELL
Connections:
- wire segments 67 -> 68
Other:
- moved on the sheet: C14, C7, D5, D6, R21

Commit message: polygons in footprint body: fix incorrect calculation of polygons with clearance or outline thickness (fix bug #1511366) Clean demos
Parts:
- C12, C6, C7, C8: footprint discret:C2 -> Discret:C2
- D5, D6, D7, D8: footprint discret:D3 -> Discret:D3
- P5, P6: footprint connect:bornier2 -> Connect:bornier2
- Q5, Q6, Q7, Q8: footprint discret:TO92-CBE -> Discret:TO92-CBE
- R10, R13, R14, R15, R16, R17, R18, R19, R21, R22, R23, R25, R26: footprint discret:R3-LARGE_PADS -> Discret:R3-LARGE_PADS
- RV2: footprint discret:RV2 -> Discret:RV2

Commit message: merge from production git:004ca3c 16.01.2017
Parts:
- U4: footprint dip_sockets:DIP-8__300_ELL -> Housings_DIP:DIP-8_W7.62mm_LongPads
Changed lines of the file:
@@
 LIBS:complex_hierarchy_schlib
 LIBS:complex_hierarchy-cache
-EELAYER 25 0
+EELAYER 26 0
 EELAYER END
 $Descr A4 11693 8268
 encoding utf-8
 Sheet 2 3
-Title ""
-Date "21 mar 2015"
-Rev ""
+Title "Complex hierarchy: demo"
+Date "2017-01-15"
+Rev "1"
 Comp ""
 Comment1 ""
@@
 AR Path="/4B3A1333/4B617B88" Ref="R26"  Part="1"
 AR Path="/4B3A13A4/4B617B88" Ref="R28"  Part="1"
-F 0 "R28" H 9200 4850 50  0000 C CNN
+F 0 "R28" V 9000 5100 50  0000 C CNN
 F 1 "220K" V 9100 5100 50  0000 C CNN
-F 2 "Discret:R3-LARGE_PADS" H 9100 5100 60  0001 C CNN
+F 2 "Discret:R3-LARGE_PADS" V 8950 5100 20  0000 C CNN
 F 3 "" H 9100 5100 60  0001 C CNN
 	1    9100 5100
@@
 F 0 "R27" V 9530 4450 50  0000 C CNN
 F 1 "47" V 9450 4450 50  0000 C CNN
-F 2 "Discret:R3-LARGE_PADS" H 9450 4450 60  0001 C CNN
+F 2 "Discret:R3-LARGE_PADS" V 9600 4450 20  0000 C CNN
 F 3 "" H 9450 4450 60  0001 C CNN
 	1    9450 4450
@@
 F 0 "D9" V 7850 4200 50  0000 C CNN
 F 1 "1N4148" V 7950 4200 50  0000 C CNN
-F 2 "Discret:D3" H 7900 4000 60  0001 C CNN
+F 2 "Discret:D3" H 7901 3929 20  0000 C CNN
 F 3 "" H 7900 4000 60  0001 C CNN
 	1    7900 4000
@@
 F 0 "R20" V 8180 5250 50  0000 C CNN
 F 1 "5,6K" V 8100 5250 50  0000 C CNN
-F 2 "Discret:R3-LARGE_PADS" H 8100 5250 60  0001 C CNN
+F 2 "Discret:R3-LARGE_PADS" V 8226 5259 20  0000 C CNN
 F 3 "" H 8100 5250 60  0001 C CNN
 	1    8100 5250
@@
 F 0 "C14" H 3000 2300 50  0000 L CNN
 F 1 "150nF" H 3000 2200 50  0000 L CNN
-F 2 "Discret:C2" H 2850 2250 60  0001 C CNN
+F 2 "Discret:C2" H 3100 2100 60  0000 C CNN
 F 3 "" H 2850 2250 60  0001 C CNN
 	1    2850 2250
@@
 F 0 "R24" V 2350 2000 50  0000 C CNN
 F 1 "1K" V 2450 2000 50  0000 C CNN
-F 2 "Discret:R3-LARGE_PADS" H 2450 2000 60  0001 C CNN
+F 2 "Discret:R3-LARGE_PADS" V 2300 2000 30  0000 C CNN
 F 3 "" H 2450 2000 60  0001 C CNN
 	1    2450 2000
@@
 F 0 "Q6" H 8500 3950 50  0000 R CNN
 F 1 "MPAS42" H 8500 3850 50  0000 R CNN
-F 2 "Discret:TO92-CBE" H 8500 3700 60  0001 C CNN
+F 2 "Discret:TO92-CBE" H 8300 3800 20  0000 C CNN
 F 3 "" H 8500 3700 60  0001 C CNN
 	1    8500 3700
@@
 F 0 "Q7" H 8500 4650 60  0000 R CNN
 F 1 "MPAS92" H 8500 4950 60  0000 R CNN
-F 2 "Discret:TO92-CBE" H 8500 4800 60  0001 C CNN
+F 2 "Discret:TO92-CBE" H 8450 5000 20  0000 C CNN
 F 3 "" H 8500 4800 60  0001 C CNN
 	1    8500 4800
@@
 F 0 "D7" V 7850 4700 50  0000 C CNN
 F 1 "1N4148" V 7950 4700 50  0000 C CNN
-F 2 "Discret:D3" H 7900 4500 60  0001 C CNN
+F 2 "Discret:D3" H 7906 4432 20  0000 C CNN
 F 3 "" H 7900 4500 60  0001 C CNN
 	1    7900 4500
@@
 F 0 "Q8" H 7800 4950 50  0000 R CNN
 F 1 "MPAS42" H 7800 5250 50  0000 R CNN
-F 2 "Discret:TO92-CBE" H 7800 5100 60  0001 C CNN
+F 2 "Discret:TO92-CBE" H 7750 4900 20  0000 C CNN
 F 3 "" H 7800 5100 60  0001 C CNN
 	1    7800 5100
@@
 F 0 "D6" V 7250 3300 50  0000 C CNN
 F 1 "1N4148" V 7350 3300 50  0000 C CNN
-F 2 "Discret:D3" H 7300 3100 60  0001 C CNN
+F 2 "Discret:D3" V 7200 3300 20  0000 C CNN
 F 3 "" H 7300 3100 60  0001 C CNN
 	1    7300 3100
@@
 F 0 "R13" V 7980 2750 50  0000 C CNN
 F 1 "470" V 7900 2750 50  0000 C CNN
-F 2 "Discret:R3-LARGE_PADS" H 7900 2750 60  0001 C CNN
+F 2 "Discret:R3-LARGE_PADS" V 8031 2758 20  0000 C CNN
 F 3 "" H 7900 2750 60  0001 C CNN
 	1    7900 2750
@@
 F 0 "D5" V 7250 3000 50  0000 C CNN
 F 1 "1N4148" V 7350 3000 50  0000 C CNN
-F 2 "Discret:D3" H 7300 2800 60  0001 C CNN
+F 2 "Discret:D3" V 7450 3000 20  0000 C CNN
 F 3 "" H 7300 2800 60  0001 C CNN
 	1    7300 2800
@@
 F 0 "R14" V 7380 3600 50  0000 C CNN
 F 1 "220K" V 7300 3600 50  0000 C CNN
-F 2 "Discret:R3-LARGE_PADS" H 7300 3600 60  0001 C CNN
+F 2 "Discret:R3-LARGE_PADS" V 7200 3600 20  0000 C CNN
 F 3 "" H 7300 3600 60  0001 C CNN
 	1    7300 3600
@@
 F 0 "R18" V 7150 5100 50  0000 C CNN
 F 1 "1K" V 7250 5100 50  0000 C CNN
-F 2 "Discret:R3-LARGE_PADS" H 7250 5100 60  0001 C CNN
+F 2 "Discret:R3-LARGE_PADS" V 7100 5100 20  0000 C CNN
 F 3 "" H 7250 5100 60  0001 C CNN
 	1    7250 5100
@@
 AR Path="/4B3A13A4/4B3A1370" Ref="R22"  Part="1"
 AR Path="/4B3A1333/4B3A1370" Ref="R12"  Part="1"
-F 0 "R22" H 9000 4850 50  0000 C CNN
+F 0 "R22" V 9000 5100 50  0000 C CNN
 F 1 "220K" V 8900 5100 50  0000 C CNN
-F 2 "Discret:R3-LARGE_PADS" H 8900 5100 60  0001 C CNN
+F 2 "Discret:R3-LARGE_PADS" V 9000 5100 20  0000 C CNN
 F 3 "" H 8900 5100 60  0001 C CNN
 	1    8900 5100
@@
 F 0 "R19" V 7300 5400 50  0000 C CNN
 F 1 "1K" V 7400 5400 50  0000 C CNN
-F 2 "Discret:R3-LARGE_PADS" H 7400 5400 60  0001 C CNN
+F 2 "Discret:R3-LARGE_PADS" V 7500 5400 30  0000 C CNN
 F 3 "" H 7400 5400 60  0001 C CNN
 	1    7400 5400
@@
 F 0 "P5" V 10700 4400 40  0000 C CNN
 F 1 "CONN_2" V 10800 4400 40  0000 C CNN
-F 2 "Connect:bornier2" H 10750 4400 60  0001 C CNN
+F 2 "Connect:bornier2" H 10750 4200 20  0000 C CNN
 F 3 "" H 10750 4400 60  0001 C CNN
 	1    10750 4400
@@
 F 0 "R16" V 3150 2000 50  0000 C CNN
 F 1 "22K" V 3250 2000 50  0000 C CNN
-F 2 "Discret:R3-LARGE_PADS" H 3250 2000 60  0001 C CNN
+F 2 "Discret:R3-LARGE_PADS" V 3100 1950 30  0000 C CNN
 F 3 "" H 3250 2000 60  0001 C CNN
 	1    3250 2000
@@
 F 0 "U4" H 6450 5600 60  0000 C CNN
 F 1 "LM358N" H 6550 5200 50  0000 C CNN
-F 2 "dip_sockets:DIP-8__300_ELL" H 6400 5400 60  0001 C CNN
+F 2 "Housings_DIP:DIP-8_W7.62mm_LongPads" H 6650 5150 20  0000 C CNN
 F 3 "" H 6400 5400 60  0001 C CNN
 	1    6400 5400
@@
 F 0 "P6" V 1300 2100 40  0000 C CNN
 F 1 "CONN_2" V 1400 2100 40  0000 C CNN
-F 2 "Connect:bornier2" H 1350 2100 60  0001 C CNN
+F 2 "Connect:bornier2" H 1300 1900 60  0000 C CNN
 F 3 "" H 1350 2100 60  0001 C CNN
 	1    1350 2100
@@
 F 0 "C7" H 4100 2650 50  0000 L CNN
 F 1 "4.7nF" H 4100 2450 50  0000 L CNN
-F 2 "Discret:C2" H 4000 2550 60  0001 C CNN
+F 2 "Discret:C2" H 4150 2400 30  0000 C CNN
 F 3 "" H 4000 2550 60  0001 C CNN
 	1    4000 2550
@@
 F 0 "C8" H 8150 5850 50  0000 L CNN
 F 1 "820pF" H 8150 5650 50  0000 L CNN
-F 2 "Discret:C2" H 8100 5750 60  0001 C CNN
+F 2 "Discret:C2" H 8268 5564 30  0000 C CNN
 F 3 "" H 8100 5750 60  0001 C CNN
 	1    8100 5750
@@
 F 0 "R15" V 9530 4150 50  0000 C CNN
 F 1 "47" V 9450 4150 50  0000 C CNN
-F 2 "Discret:R3-LARGE_PADS" H 9450 4150 60  0001 C CNN
+F 2 "Discret:R3-LARGE_PADS" V 9400 4150 20  0000 C CNN
 F 3 "" H 9450 4150 60  0001 C CNN
 	1    9450 4150
@@
 F 0 "R21" V 5150 6400 50  0000 C CNN
 F 1 "4,7K" V 5250 6400 50  0000 C CNN
-F 2 "Discret:R3-LARGE_PADS" H 5250 6400 60  0001 C CNN
+F 2 "Discret:R3-LARGE_PADS" V 5100 6400 30  0000 C CNN
 F 3 "" H 5250 6400 60  0001 C CNN
 	1    5250 6400
@@
 F 0 "Q5" H 7800 3150 60  0000 R CNN
 F 1 "MPAS92" H 7800 3450 60  0000 R CNN
-F 2 "Discret:TO92-CBE" H 7800 3300 60  0001 C CNN
+F 2 "Discret:TO92-CBE" H 7750 3100 20  0000 C CNN
 F 3 "" H 7800 3300 60  0001 C CNN
 	1    7800 3300
@@
 F 0 "U4" H 4900 2600 60  0000 C CNN
 F 1 "LM358N" H 5000 2200 50  0000 C CNN
-F 2 "dip_sockets:DIP-8__300_ELL" H 4850 2400 60  0001 C CNN
+F 2 "Housings_DIP:DIP-8_W7.62mm_LongPads" H 5100 2150 20  0000 C CNN
 F 3 "" H 4850 2400 60  0001 C CNN
 	2    4850 2400
@@
 F 0 "R17" V 3850 2000 50  0000 C CNN
 F 1 "22K" V 3950 2000 50  0000 C CNN
-F 2 "Discret:R3-LARGE_PADS" H 3950 2000 60  0001 C CNN
+F 2 "Discret:R3-LARGE_PADS" V 3800 2000 30  0000 C CNN
 F 3 "" H 3950 2000 60  0001 C CNN
 	1    3950 2000
@@
 F 0 "C6" V 4200 1600 50  0000 C CNN
 F 1 "15nF" V 4500 1600 50  0000 C CNN
-F 2 "Discret:C2" H 4350 1600 60  0001 C CNN
+F 2 "Discret:C2" V 4100 1600 60  0000 C CNN
 F 3 "" H 4350 1600 60  0001 C CNN
 	1    4350 1600
 	0    1    1    0
 $EndComp
-Text Notes 3100 2900 0    60   ~ 0
+Text Notes 2600 2950 0    80   Italic 16
 Filter:\nFc =1000Hz
 $Comp
@@
 F 0 "RV2" H 5850 6300 50  0000 C CNN
 F 1 "4,7K" H 5850 6400 50  0000 C CNN
-F 2 "Discret:RV2" H 5850 6400 60  0001 C CNN
+F 2 "Discret:RV2" H 5850 6250 30  0000 C CNN
 F 3 "" H 5850 6400 60  0001 C CNN
 	1    5850 6400
