File: demos/complex_hierarchy/complex_hierarchy.kicad_pcb (KiCad board)
At the start: 2 copper layers, 100.3 x 80 mm, 68 parts, among them P1 CONN_2, P2 CONN_2, P3 CONN_2, P4 CONN_2, P5 CONN_2, P6 CONN_2, Q1 MPAS92, Q2 MPAS42, Q3 MPAS92, Q4 MPAS42, Q5 MPAS92, Q6 MPAS42, Q7 MPAS92, Q8 MPAS42, U1 ICL7660, U2 78L05, U3 LM358N, U4 LM358N

Commit message: merge from production git:004ca3c 16.01.2017
Parts:
- C1, C10, C11, C2: footprint discret:CP6 -> Discret:CP6
- C12, C14, C3, C4, C5, C6, C7, C8: footprint discret:C2 -> Discret:C2
- C9: footprint discret:CP8 -> Discret:CP8
- D1: footprint discret:D5 -> Discret:D5
- D2, D3, D4, D5, D6, D7, D8, D9: footprint discret:D3 -> Discret:D3
- P1, P2, P3, P4, P5, P6: footprint connect:bornier2 -> Connect:bornier2
- Q1, Q2, Q3, Q4, Q5, Q6, Q7, Q8: footprint discret:TO92-CBE -> Discret:TO92-CBE
- R10, R11, R12, R13, R14, R15, R16, R17, R18, R19, R20, R21, R22, R23, R24, R25, R26, R27, R28, R3, R4, R5, R6, R7, R8, R9: footprint discret:R3-LARGE_PADS -> Discret:R3-LARGE_PADS
- RV1, RV2: footprint discret:RV2 -> Discret:RV2
- U1, U3, U4: footprint dip_sockets:DIP-8__300_ELL -> Housings_DIP:DIP-8_W7.62mm_LongPads
- U2: footprint discret:LM78LXX -> Discret:LM78LXX
- moved U1 5.39 mm to (145.4, 72.1), turned to 90 degrees
- moved U3 5.39 mm to (107.3, 124.2), turned to 90 degrees
- moved U4 5.39 mm to (107.3, 96.3), turned to 90 degrees
Other:
- board text added: "Complex hierarchy Demo"
- board text removed: "Actionneur Piezo New Amp V02"
